File: ActivePrecharge.kicad_sch (KiCad schematic)
At the start: 36 parts, among them Q2 PMV20XNER, Q3 PMV20XNER, U1 TLV9301xDCK, U2 TLV9301xDCK, U4 TCMT1106, U5 TCMT1106

Commit message: sch additions
Connections:
- net AVef is gone; now on net AVref: Q3.1 (G)
- net MPre- is gone; now on net MVin: R3.1
- net MVin: no longer AIn_TP1.1, C4.1, R7.2, R9.2, U2.3 (-)
- net APre+ renamed AVref
- net AVref: now also ARef_TP1.1, C3.1, R10.2, R6.2, R8.2, U2.1 (+)
- net APre- renamed AVin
- net AVin: now also AIn_TP1.1, C4.1, R7.2, R9.2, U2.3 (-)
- net MPre+ renamed MVref
- net MVref: now also C1.1, MRef_TP1.1, Q2.1 (G), R1.2, R2.2, R5.2, U1.1 (+)
- removed net MVef: ARef_TP1.1, C1.1, C3.1, MRef_TP1.1, Q2.1 (G), R1.2, R10.2, R2.2, R5.2, R6.2, R8.2, U1.1 (+), U2.1 (+)
Changed lines of the file:
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@@
 		)
 	)
-	(label "AVef"
+	(label "AVref"
 		(at 144.78 110.49 0)
 		(effects
@@
 		)
 	)
-	(label "MVef"
+	(label "MVref"
 		(at 144.78 45.72 0)
 		(effects
@@
 		)
 	)
-	(label "MVin"
+	(label "AVin"
 		(at 92.71 128.27 0)
 		(effects
@@
 		)
 	)
-	(label "MVef"
+	(label "AVref"
 		(at 92.71 120.65 0)
 		(effects
@@
 		)
 	)
-	(label "MVef"
+	(label "MVref"
 		(at 92.71 55.88 0)
 		(effects
@@
 		)
 	)
-	(hierarchical_label "MPre-"
+	(hierarchical_label "MVin"
 		(shape input)
 		(at 54.61 63.5 180)
@@
 		)
 	)
-	(hierarchical_label "APre-"
+	(hierarchical_label "AVin"
 		(shape input)
 		(at 54.61 128.27 180)
@@
 		)
 	)
-	(hierarchical_label "MPre+"
+	(hierarchical_label "MVref"
 		(shape input)
 		(at 54.61 40.64 180)
@@
 		)
 	)
-	(hierarchical_label "APre+"
+	(hierarchical_label "AVref"
 		(shape input)
 		(at 54.61 105.41 180)
