File: HVArchitecture.kicad_sch (KiCad schematic)
At the start: 6 parts, among them J3 Conn_01x02, Q1 Q_PMOS_GDS

Commit message: sch additions
Parts:
- removed 12V_TP1, LVGND_TP1: TestPoint, utsvt-special:TestPoint_HEX_3mmID, symbol Connector:TestPoint
- removed D1: BZT52-B12-QX, Active-PrechargeLib:BZT52B12QX, symbol Device:D_Zener
- removed J3: Conn_01x02, utsvt-conn:Molex_MicroFit3.0_1x2xP3.00mm_PolarizingPeg_Vertical, symbol Connector_Generic:Conn_01x02
- removed Q1: Q_PMOS_GDS, Package_TO_SOT_SMD:SOT-23-3, symbol Device:Q_PMOS_GDS
- removed R11: 49.9k, Resistor_SMD:R_0805_2012Metric, symbol Device:R_US
- added C101: 270u, symbol Device:C
- added C102: 440u, symbol Device:C_Polarized_US
- added D2, D3, D4, D5, D6, D7: RSX068MP2STR, Diode_SMD:D_SOD-123F, symbol Device:D_Schottky
- added F1, F2, F3, F4: Fuse, Fuse:Fuseholder_Blade_Mini_Keystone_3568, symbol Device:Fuse
- added HVGND1: TestPoint, utsvt-special:TestPoint_HEX_3mmID, symbol Connector:TestPoint
- added J1, J2: Conn_01x03, utsvt-conn:Molex_MicroFit3.0_1x3xP3.00mm_PolarizingPeg_Vertical, symbol Connector_Generic:Conn_01x03
- added R101, R102: 750, symbol Device:R_US
Connections:
- net HVGND: now also C101.2, C102.2, D2.2 (A), D7.2 (A), HVGND1.1
- new net: D6.2 (A), F4.2
- new net: D5.2 (A), F3.2
- new net: D4.2 (A), F2.2
- new net: D3.2 (A), F1.2
- new net APre+: F3.1, J2.1 (Pin_1), R102.1
- new net APre-: C102.1, F4.1, J2.3 (Pin_3), R102.2
- new net AVin: D5.1 (K)
- new net AVref: D6.1 (K)
- new net A_HVGND: D2.1 (K), J2.2 (Pin_2)
- new net HGND: D7.1 (K), J1.2 (Pin_2)
- new net MPre+: F2.1, J1.3 (Pin_3), R101.1
- new net MPre-: C101.1, F1.1, J1.1 (Pin_1), R101.2
- new net MVin: D3.1 (K)
- new net MVref: D4.1 (K)
Other:
- removed sheet ActivePrecharge
- removed sheet CAN
- removed sheet ContactorDriver
- removed sheet HVArchitecture
- removed sheet PowerMisc
- note added: "Array Precharge Reisitor"
- note added: "Excluded from board"
- note added: "MOCO Bulk Cap"
- note added: "MPPT Bulk Cap"
- note added: "Motor Precharge Reisitor"
