File: Buttond_LEDs_IO.kicad_sch (KiCad schematic)
At the start: 15 parts, among them J13 IO_Breakout, SW1 RESET, SW2 BOOT

Commit message: added opto's to sense signals
Parts:
- C1, C2: footprint (none) -> Capacitor_SMD:C_0805_2012Metric
- R1, R2: footprint (none) -> Resistor_SMD:R_0805_2012Metric
Changed lines of the file:
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@@
 			)
 		)
-		(property "Footprint" ""
+		(property "Footprint" "Capacitor_SMD:C_0805_2012Metric"
 			(at 59.9948 72.39 0)
 			(effects
@@
 			)
 		)
-		(property "Footprint" ""
+		(property "Footprint" "Resistor_SMD:R_0805_2012Metric"
 			(at 59.944 56.134 90)
 			(effects
@@
 			)
 		)
-		(property "Footprint" ""
+		(property "Footprint" "Resistor_SMD:R_0805_2012Metric"
 			(at 59.944 98.044 90)
 			(effects
@@
 			)
 		)
-		(property "Footprint" ""
+		(property "Footprint" "Capacitor_SMD:C_0805_2012Metric"
 			(at 59.9948 114.3 0)
 			(effects

Commit message: layout start
Parts:
- J16: renamed from J13; footprint (none) -> Connector_PinHeader_2.54mm:PinHeader_1x04_P2.54mm_Vertical
- SW1, SW2: footprint (none) -> UTSVT_Special:SW_SPST_B3SL-1002P
- renumbered C1 to C15, C2 to C16, R1 to R25, R2 to R26, R35 to R27, R36 to R28, R37 to R29, R38 to R30
Connections:
- net BOOT: now also SW2.2 (A); no longer SW2.3 (B)
- net Reset: now also SW1.2 (A); no longer SW1.3 (B)
Changed lines of the file:
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@@
 		(dnp no)
 		(fields_autoplaced yes)
-		(property "Reference" "#PWR052"
+		(property "Reference" "#PWR051"
 			(at 156.21 107.95 0)
 			(effects
@@
 			(project "VehicleControlUnit"
 				(path "/795c8e51-3ded-4d21-b864-aaff31c5def7/6282503b-e4ab-454b-a074-f701a067f39b/cecfe08a-2de2-4171-9051-c68b429ab9e8"
-					(reference "#PWR052")
+					(reference "#PWR051")
 					(unit 1)
 				)
@@
 			)
 		)
-		(property "Footprint" ""
+		(property "Footprint" "UTSVT_Special:SW_SPST_B3SL-1002P"
 			(at 71.12 100.33 0)
 			(effects
@@
 			)
 		)
-		(pin "3"
+		(pin "2"
 		)
 		(pin "4"
@@
 		(dnp no)
 		(fields_autoplaced yes)
-		(property "Reference" "R35"
+		(property "Reference" "R27"
 			(at 135.89 82.5499 0)
 			(effects
@@
 			(project "VehicleControlUnit"
 				(path "/795c8e51-3ded-4d21-b864-aaff31c5def7/6282503b-e4ab-454b-a074-f701a067f39b/cecfe08a-2de2-4171-9051-c68b429ab9e8"
-					(reference "R35")
+					(reference "R27")
 					(unit 1)
 				)
@@
 		(dnp no)
 		(fields_autoplaced yes)
-		(property "Reference" "#PWR024"
+		(property "Reference" "#PWR046"
 			(at 60.96 121.92 0)
 			(effects
@@
 			(project "VehicleControlUnit"
 				(path "/795c8e51-3ded-4d21-b864-aaff31c5def7/6282503b-e4ab-454b-a074-f701a067f39b/cecfe08a-2de2-4171-9051-c68b429ab9e8"
-					(reference "#PWR024")
+					(reference "#PWR046")
 					(unit 1)
 				)
@@
 		(dnp no)
 		(fields_autoplaced yes)
-		(property "Reference" "#PWR053"
+		(property "Reference" "#PWR052"
 			(at 167.64 107.95 0)
 			(effects
@@
 			(project "VehicleControlUnit"
 				(path "/795c8e51-3ded-4d21-b864-aaff31c5def7/6282503b-e4ab-454b-a074-f701a067f39b/cecfe08a-2de2-4171-9051-c68b429ab9e8"
-					(reference "#PWR053")
+					(reference "#PWR052")
 					(unit 1)
 				)
@@
 		(dnp no)
 		(fields_autoplaced yes)
-		(property "Reference" "C1"
+		(property "Reference" "C15"
 			(at 57.15 67.3099 0)
 			(effects
@@
 			(project "VehicleControlUnit"
 				(path "/795c8e51-3ded-4d21-b864-aaff31c5def7/6282503b-e4ab-454b-a074-f701a067f39b/cecfe08a-2de2-4171-9051-c68b429ab9e8"
-					(reference "C1")
+					(reference "C15")
 					(unit 1)
 				)
@@
 		(dnp no)
 		(fields_autoplaced yes)
-		(property "Reference" "#PWR04"
+		(property "Reference" "#PWR045"
 			(at 60.96 80.01 0)
 			(effects
@@
 			(project "VehicleControlUnit"
 				(path "/795c8e51-3ded-4d21-b864-aaff31c5def7/6282503b-e4ab-454b-a074-f701a067f39b/cecfe08a-2de2-4171-9051-c68b429ab9e8"
-					(reference "#PWR04")
+					(reference "#PWR045")
 					(unit 1)
 				)
@@
 		(dnp no)
 		(fields_autoplaced yes)
-		(property "Reference" "R1"
+		(property "Reference" "R25"
 			(at 58.42 54.6099 0)
 			(effects
@@
 			(project "VehicleControlUnit"
 				(path "/795c8e51-3ded-4d21-b864-aaff31c5def7/6282503b-e4ab-454b-a074-f701a067f39b/cecfe08a-2de2-4171-9051-c68b429ab9e8"
-					(reference "R1")
+					(reference "R25")
 					(unit 1)
 				)
@@
 		(dnp no)
 		(fields_autoplaced yes)
-		(property "Reference" "R36"
+		(property "Reference" "R28"
 			(at 147.32 82.5499 0)
 			(effects
@@
 			(project "VehicleControlUnit"
 				(path "/795c8e51-3ded-4d21-b864-aaff31c5def7/6282503b-e4ab-454b-a074-f701a067f39b/cecfe08a-2de2-4171-9051-c68b429ab9e8"
-					(reference "R36")
+					(reference "R28")
 					(unit 1)
 				)
@@
 		(dnp no)
 		(fields_autoplaced yes)
-		(property "Reference" "#PWR02"
+		(property "Reference" "#PWR047"
 			(at 80.01 80.01 0)
 			(effects
@@
 			(project "VehicleControlUnit"
 				(path "/795c8e51-3ded-4d21-b864-aaff31c5def7/6282503b-e4ab-454b-a074-f701a067f39b/cecfe08a-2de2-4171-9051-c68b429ab9e8"
-					(reference "#PWR02")
+					(reference "#PWR047")
 					(unit 1)
 				)
@@
 		(dnp no)
 		(fields_autoplaced yes)
-		(property "Reference" "R37"
+		(property "Reference" "R29"
 			(at 158.75 82.5499 0)
 			(effects
@@
 			(project "VehicleControlUnit"
 				(path "/795c8e51-3ded-4d21-b864-aaff31c5def7/6282503b-e4ab-454b-a074-f701a067f39b/cecfe08a-2de2-4171-9051-c68b429ab9e8"
-					(reference "R37")
+					(reference "R29")
 					(unit 1)
 				)
@@
 		(dnp no)
 		(fields_autoplaced yes)
-		(property "Reference" "#PWR050"
+		(property "Reference" "#PWR049"
 			(at 133.35 107.95 0)
 			(effects
@@
 			(project "VehicleControlUnit"
 				(path "/795c8e51-3ded-4d21-b864-aaff31c5def7/6282503b-e4ab-454b-a074-f701a067f39b/cecfe08a-2de2-4171-9051-c68b429ab9e8"
-					(reference "#PWR050")
+					(reference "#PWR049")
 					(unit 1)
 				)
@@
 		(dnp no)
 		(fields_autoplaced yes)
-		(property "Reference" "R38"
+		(property "Reference" "R30"
 			(at 170.18 82.5499 0)
 			(effects
@@
 			(project "VehicleControlUnit"
 				(path "/795c8e51-3ded-4d21-b864-aaff31c5def7/6282503b-e4ab-454b-a074-f701a067f39b/cecfe08a-2de2-4171-9051-c68b429ab9e8"
-					(reference "R38")
-					(unit 1)
-				)
-			)
-		)
-	)
-	(symbol
+					(reference "R30")
+					(unit 1)
+				)
+			)
+		)
+	)
+	(symbol
+		(lib_name "SW_MEC_5G_1")
 		(lib_id "Switch:SW_MEC_5G")
 		(at 71.12 63.5 0)
@@
 			)
 		)
-		(property "Footprint" ""
+		(property "Footprint" "UTSVT_Special:SW_SPST_B3SL-1002P"
 			(at 71.12 58.42 0)
 			(effects
@@
 			)
 		)
-		(pin "3"
+		(pin "2"
 		)
 		(pin "4"
@@
 		(dnp no)
 		(fields_autoplaced yes)
-		(property "Reference" "#PWR05"
+		(property "Reference" "#PWR048"
 			(at 80.01 121.92 0)
 			(effects
@@
 			(project "VehicleControlUnit"
 				(path "/795c8e51-3ded-4d21-b864-aaff31c5def7/6282503b-e4ab-454b-a074-f701a067f39b/cecfe08a-2de2-4171-9051-c68b429ab9e8"
-					(reference "#PWR05")
+					(reference "#PWR048")
 					(unit 1)
 				)
@@
 		(dnp no)
 		(fields_autoplaced yes)
-		(property "Reference" "#PWR051"
+		(property "Reference" "#PWR050"
 			(at 144.78 107.95 0)
 			(effects
@@
 			(project "VehicleControlUnit"
 				(path "/795c8e51-3ded-4d21-b864-aaff31c5def7/6282503b-e4ab-454b-a074-f701a067f39b/cecfe08a-2de2-4171-9051-c68b429ab9e8"
-					(reference "#PWR051")
+					(reference "#PWR050")
 					(unit 1)
 				)
@@
 		(dnp no)
 		(fields_autoplaced yes)
-		(property "Reference" "R2"
+		(property "Reference" "R26"
 			(at 58.42 96.5199 0)
 			(effects
@@
 			(project "VehicleControlUnit"
 				(path "/795c8e51-3ded-4d21-b864-aaff31c5def7/6282503b-e4ab-454b-a074-f701a067f39b/cecfe08a-2de2-4171-9051-c68b429ab9e8"
-					(reference "R2")
+					(reference "R26")
 					(unit 1)
 				)
@@
 		(dnp no)
 		(fields_autoplaced yes)
-		(property "Reference" "C2"
+		(property "Reference" "C16"
 			(at 57.15 109.2199 0)
 			(effects
@@
 			(project "VehicleControlUnit"
 				(path "/795c8e51-3ded-4d21-b864-aaff31c5def7/6282503b-e4ab-454b-a074-f701a067f39b/cecfe08a-2de2-4171-9051-c68b429ab9e8"
-					(reference "C2")
+					(reference "C16")
 					(unit 1)
 				)
@@
 		(dnp no)
 		(fields_autoplaced yes)
-		(property "Reference" "J13"
+		(property "Reference" "J16"
 			(at 248.92 85.0899 0)
 			(effects
@@
 			)
 		)
-		(property "Footprint" ""
+		(property "Footprint" "Connector_PinHeader_2.54mm:PinHeader_1x04_P2.54mm_Vertical"
 			(at 246.38 85.09 0)
 			(effects
@@
 			(project ""
 				(path "/795c8e51-3ded-4d21-b864-aaff31c5def7/6282503b-e4ab-454b-a074-f701a067f39b/cecfe08a-2de2-4171-9051-c68b429ab9e8"
-					(reference "J13")
-					(unit 1)
-				)
+					(reference "J16")
+					(unit 1)
+				)

Commit message: first revision
Parts:
- added J17: IO_5-8, Connector_PinHeader_2.54mm:PinHeader_1x04_P2.54mm_Vertical, symbol Connector_Generic:Conn_01x04
- added J18: IO_9-12, Connector_PinHeader_2.54mm:PinHeader_1x04_P2.54mm_Vertical, symbol Connector_Generic:Conn_01x04
- J16: value IO_Breakout -> IO_1-4
- renumbered C15 to C16, C16 to C17
Connections:
- net BOOT: no longer SW2.4 (B)
- net GND: no longer SW1.2 (A), SW2.2 (A)
- net Reset: no longer SW1.4 (B)
- new net IO10: J18.2 (Pin_2)
- new net IO11: J18.3 (Pin_3)
- new net IO12: J18.4 (Pin_4)
- new net IO5: J17.1 (Pin_1)
- new net IO6: J17.2 (Pin_2)
- new net IO7: J17.3 (Pin_3)
- new net IO8: J17.4 (Pin_4)
- new net IO9: J18.1 (Pin_1)

Commit message: tweaking
Other:
- moved on the sheet: J16, J17, J18
Changed lines of the file:
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@@
 	(wire
 		(pts
-			(xy 237.49 111.76) (xy 241.3 111.76)
-		)
-		(stroke
-			(width 0)
-			(type default)
-		)
-	)
-	(wire
-		(pts
-			(xy 237.49 94.615) (xy 241.3 94.615)
+			(xy 235.585 112.395) (xy 239.395 112.395)
+		)
+		(stroke
+			(width 0)
+			(type default)
+		)
+	)
+	(wire
+		(pts
+			(xy 235.585 84.455) (xy 239.395 84.455)
 		)
 		(stroke
@@
 	(wire
 		(pts
-			(xy 237.49 102.235) (xy 241.3 102.235)
+			(xy 235.585 92.075) (xy 239.395 92.075)
 		)
 		(stroke
@@
 	(wire
 		(pts
-			(xy 237.49 114.3) (xy 241.3 114.3)
-		)
-		(stroke
-			(width 0)
-			(type default)
-		)
-	)
-	(wire
-		(pts
-			(xy 237.49 82.55) (xy 241.3 82.55)
+			(xy 235.585 114.935) (xy 239.395 114.935)
+		)
+		(stroke
+			(width 0)
+			(type default)
+		)
+	)
+	(wire
+		(pts
+			(xy 235.585 62.23) (xy 239.395 62.23)
 		)
 		(stroke
@@
 	(wire
 		(pts
-			(xy 237.49 99.695) (xy 241.3 99.695)
+			(xy 235.585 89.535) (xy 239.395 89.535)
 		)
 		(stroke
@@
 	(wire
 		(pts
-			(xy 237.49 109.22) (xy 241.3 109.22)
+			(xy 235.585 109.855) (xy 239.395 109.855)
 		)
 		(stroke
@@
 	(wire
 		(pts
-			(xy 237.49 106.68) (xy 241.3 106.68)
+			(xy 235.585 107.315) (xy 239.395 107.315)
 		)
 		(stroke
@@
 	(wire
 		(pts
-			(xy 237.49 97.155) (xy 241.3 97.155)
+			(xy 235.585 86.995) (xy 239.395 86.995)
 		)
 		(stroke
@@
 	(wire
 		(pts
-			(xy 237.49 90.17) (xy 241.3 90.17)
+			(xy 235.585 69.85) (xy 239.395 69.85)
 		)
 		(stroke
@@
 	(wire
 		(pts
-			(xy 237.49 87.63) (xy 241.3 87.63)
+			(xy 235.585 67.31) (xy 239.395 67.31)
 		)
 		(stroke
@@
 	(wire
 		(pts
-			(xy 237.49 85.09) (xy 241.3 85.09)
+			(xy 235.585 64.77) (xy 239.395 64.77)
 		)
 		(stroke
@@
 	(hierarchical_label "IO5"
 		(shape input)
-		(at 237.49 94.615 180)
+		(at 235.585 84.455 180)
 		(effects
 			(font
@@
 	(hierarchical_label "IO4"
 		(shape input)
-		(at 237.49 90.17 180)
+		(at 235.585 69.85 180)
 		(effects
 			(font
@@
 	(hierarchical_label "IO10"
 		(shape input)
-		(at 237.49 109.22 180)
+		(at 235.585 109.855 180)
 		(effects
 			(font
@@
 	(hierarchical_label "IO7"
 		(shape input)
-		(at 237.49 99.695 180)
+		(at 235.585 89.535 180)
 		(effects
 			(font
@@
 	(hierarchical_label "IO9"
 		(shape input)
-		(at 237.49 106.68 180)
+		(at 235.585 107.315 180)
 		(effects
 			(font
@@
 	(hierarchical_label "IO6"
 		(shape input)
-		(at 237.49 97.155 180)
+		(at 235.585 86.995 180)
 		(effects
 			(font
@@
 	(hierarchical_label "IO2"
 		(shape input)
-		(at 237.49 85.09 180)
+		(at 235.585 64.77 180)
 		(effects
 			(font
@@
 	(hierarchical_label "IO1"
 		(shape input)
-		(at 237.49 82.55 180)
+		(at 235.585 62.23 180)
 		(effects
 			(font
@@
 	(hierarchical_label "IO12"
 		(shape input)
-		(at 237.49 114.3 180)
+		(at 235.585 114.935 180)
 		(effects
 			(font
@@
 	(hierarchical_label "IO3"
 		(shape input)
-		(at 237.49 87.63 180)
+		(at 235.585 67.31 180)
 		(effects
 			(font
@@
 	(hierarchical_label "IO11"
 		(shape input)
-		(at 237.49 111.76 180)
+		(at 235.585 112.395 180)
 		(effects
 			(font
@@
 	(hierarchical_label "IO8"
 		(shape input)
-		(at 237.49 102.235 180)
+		(at 235.585 92.075 180)
 		(effects
 			(font
@@
 	(symbol
 		(lib_id "Connector_Generic:Conn_01x04")
-		(at 246.38 97.155 0)
+		(at 244.475 86.995 0)
 		(unit 1)
 		(exclude_from_sim no)
@@
 		(fields_autoplaced yes)
 		(property "Reference" "J17"
-			(at 248.92 97.1549 0)
+			(at 247.015 86.9949 0)
 			(effects
 				(font
@@
 		)
 		(property "Value" "IO_5-8"
-			(at 248.92 99.6949 0)
+			(at 247.015 89.5349 0)
 			(effects
 				(font
@@
 		)
 		(property "Footprint" "Connector_PinHeader_2.54mm:PinHeader_1x04_P2.54mm_Vertical"
-			(at 246.38 97.155 0)
+			(at 244.475 86.995 0)
 			(effects
 				(font
@@
 		)
 		(property "Datasheet" "~"
-			(at 246.38 97.155 0)
+			(at 244.475 86.995 0)
 			(effects
 				(font
@@
 		)
 		(property "Description" "Generic connector, single row, 01x04, script generated (kicad-library-utils/schlib/autogen/connector/)"
-			(at 246.38 97.155 0)
+			(at 244.475 86.995 0)
 			(effects
 				(font
@@
 	(symbol
 		(lib_id "Connector_Generic:Conn_01x04")
-		(at 246.38 109.22 0)
+		(at 244.475 109.855 0)
 		(unit 1)
 		(exclude_from_sim no)
@@
 		(fields_autoplaced yes)
 		(property "Reference" "J18"
-			(at 248.92 109.2199 0)
+			(at 247.015 109.8549 0)
 			(effects
 				(font
@@
 		)
 		(property "Value" "IO_9-12"
-			(at 248.92 111.7599 0)
+			(at 247.015 112.3949 0)
 			(effects
 				(font
@@
 		)
 		(property "Footprint" "Connector_PinHeader_2.54mm:PinHeader_1x04_P2.54mm_Vertical"
-			(at 246.38 109.22 0)
+			(at 244.475 109.855 0)
 			(effects
 				(font
@@
 		)
 		(property "Datasheet" "~"
-			(at 246.38 109.22 0)
+			(at 244.475 109.855 0)
 			(effects
 				(font
@@
 		)
 		(property "Description" "Generic connector, single row, 01x04, script generated (kicad-library-utils/schlib/autogen/connector/)"
-			(at 246.38 109.22 0)
+			(at 244.475 109.855 0)
 			(effects
 				(font
@@
 	(symbol
 		(lib_id "Connector_Generic:Conn_01x04")
-		(at 246.38 85.09 0)
+		(at 244.475 64.77 0)
 		(unit 1)
 		(exclude_from_sim no)
@@
 		(fields_autoplaced yes)
 		(property "Reference" "J16"
-			(at 248.92 85.0899 0)
+			(at 247.015 64.7699 0)
 			(effects
 				(font
@@
 		)
 		(property "Value" "IO_1-4"
-			(at 248.92 87.6299 0)
+			(at 247.015 67.3099 0)
 			(effects
 				(font
@@
 		)
 		(property "Footprint" "Connector_PinHeader_2.54mm:PinHeader_1x04_P2.54mm_Vertical"
-			(at 246.38 85.09 0)
+			(at 244.475 64.77 0)
 			(effects
 				(font
@@
 		)
 		(property "Datasheet" "~"
-			(at 246.38 85.09 0)
+			(at 244.475 64.77 0)
 			(effects
 				(font
@@
 		)
 		(property "Description" "Generic connector, single row, 01x04, script generated (kicad-library-utils/schlib/autogen/connector/)"
-			(at 246.38 85.09 0)
-			(effects
-				(font
+			(at 244.475 64.77 0)
+			(effects
+				(font

Commit message: fixed
Parts:
- removed J17: IO_5-8, Connector_PinHeader_2.54mm:PinHeader_1x04_P2.54mm_Vertical, symbol Connector_Generic:Conn_01x04
- removed J18: IO_9-12, Connector_PinHeader_2.54mm:PinHeader_1x04_P2.54mm_Vertical, symbol Connector_Generic:Conn_01x04
- added J17: Conn_01x08, Connector_PinHeader_2.54mm:PinHeader_1x08_P2.54mm_Vertical, symbol Connector_Generic:Conn_01x08
- J16: value IO_1-4 -> Conn_01x04
- renumbered C16 to C15, C17 to C16
Connections:
- net IO10: now also J17.6 (Pin_6)
- net IO11: now also J17.7 (Pin_7)
- net IO12: now also J17.8 (Pin_8)
- net IO5: now also J17.1 (Pin_1)
- net IO6: now also J17.2 (Pin_2)
- net IO7: now also J17.3 (Pin_3)
- net IO8: now also J17.4 (Pin_4)
- net IO9: now also J17.5 (Pin_5)

Commit message: review changes
Parts:
- renumbered J16 to J15, J17 to J16
Changed lines of the file:
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@@
 		(dnp no)
 		(fields_autoplaced yes)
-		(property "Reference" "J17"
+		(property "Reference" "J16"
 			(at 247.65 90.8049 0)
 			(effects
@@
 			(project ""
 				(path "/795c8e51-3ded-4d21-b864-aaff31c5def7/6282503b-e4ab-454b-a074-f701a067f39b/cecfe08a-2de2-4171-9051-c68b429ab9e8"
-					(reference "J17")
+					(reference "J16")
 					(unit 1)
 				)
@@
 		(dnp no)
 		(fields_autoplaced yes)
-		(property "Reference" "#PWR045"
+		(property "Reference" "#PWR062"
 			(at 156.21 107.95 0)
 			(effects
@@
 			(project "VehicleControlUnit"
 				(path "/795c8e51-3ded-4d21-b864-aaff31c5def7/6282503b-e4ab-454b-a074-f701a067f39b/cecfe08a-2de2-4171-9051-c68b429ab9e8"
-					(reference "#PWR045")
+					(reference "#PWR062")
 					(unit 1)
 				)
@@
 		(dnp no)
 		(fields_autoplaced yes)
-		(property "Reference" "J16"
+		(property "Reference" "J15"
 			(at 247.65 62.8649 0)
 			(effects
@@
 			(project ""
 				(path "/795c8e51-3ded-4d21-b864-aaff31c5def7/6282503b-e4ab-454b-a074-f701a067f39b/cecfe08a-2de2-4171-9051-c68b429ab9e8"
-					(reference "J16")
+					(reference "J15")
 					(unit 1)
 				)
@@
 		(dnp no)
 		(fields_autoplaced yes)
-		(property "Reference" "#PWR040"
+		(property "Reference" "#PWR057"
 			(at 60.96 121.92 0)
 			(effects
@@
 			(project "VehicleControlUnit"
 				(path "/795c8e51-3ded-4d21-b864-aaff31c5def7/6282503b-e4ab-454b-a074-f701a067f39b/cecfe08a-2de2-4171-9051-c68b429ab9e8"
-					(reference "#PWR040")
+					(reference "#PWR057")
 					(unit 1)
 				)
@@
 		(dnp no)
 		(fields_autoplaced yes)
-		(property "Reference" "#PWR046"
+		(property "Reference" "#PWR063"
 			(at 167.64 107.95 0)
 			(effects
@@
 			(project "VehicleControlUnit"
 				(path "/795c8e51-3ded-4d21-b864-aaff31c5def7/6282503b-e4ab-454b-a074-f701a067f39b/cecfe08a-2de2-4171-9051-c68b429ab9e8"
-					(reference "#PWR046")
+					(reference "#PWR063")
 					(unit 1)
 				)
@@
 		(dnp no)
 		(fields_autoplaced yes)
-		(property "Reference" "#PWR039"
+		(property "Reference" "#PWR056"
 			(at 60.96 80.01 0)
 			(effects
@@
 			(project "VehicleControlUnit"
 				(path "/795c8e51-3ded-4d21-b864-aaff31c5def7/6282503b-e4ab-454b-a074-f701a067f39b/cecfe08a-2de2-4171-9051-c68b429ab9e8"
-					(reference "#PWR039")
+					(reference "#PWR056")
 					(unit 1)
 				)
@@
 		(dnp no)
 		(fields_autoplaced yes)
-		(property "Reference" "#PWR041"
+		(property "Reference" "#PWR058"
 			(at 80.01 80.01 0)
 			(effects
@@
 			(project "VehicleControlUnit"
 				(path "/795c8e51-3ded-4d21-b864-aaff31c5def7/6282503b-e4ab-454b-a074-f701a067f39b/cecfe08a-2de2-4171-9051-c68b429ab9e8"
-					(reference "#PWR041")
+					(reference "#PWR058")
 					(unit 1)
 				)
@@
 		(dnp no)
 		(fields_autoplaced yes)
-		(property "Reference" "#PWR043"
+		(property "Reference" "#PWR060"
 			(at 133.35 107.95 0)
 			(effects
@@
 			(project "VehicleControlUnit"
 				(path "/795c8e51-3ded-4d21-b864-aaff31c5def7/6282503b-e4ab-454b-a074-f701a067f39b/cecfe08a-2de2-4171-9051-c68b429ab9e8"
-					(reference "#PWR043")
+					(reference "#PWR060")
 					(unit 1)
 				)
@@
 		(dnp no)
 		(fields_autoplaced yes)
-		(property "Reference" "#PWR042"
+		(property "Reference" "#PWR059"
 			(at 80.01 121.92 0)
 			(effects
@@
 			(project "VehicleControlUnit"
 				(path "/795c8e51-3ded-4d21-b864-aaff31c5def7/6282503b-e4ab-454b-a074-f701a067f39b/cecfe08a-2de2-4171-9051-c68b429ab9e8"
-					(reference "#PWR042")
+					(reference "#PWR059")
 					(unit 1)
 				)
@@
 		(dnp no)
 		(fields_autoplaced yes)
-		(property "Reference" "#PWR044"
+		(property "Reference" "#PWR061"
 			(at 144.78 107.95 0)
 			(effects
@@
 			(project "VehicleControlUnit"
 				(path "/795c8e51-3ded-4d21-b864-aaff31c5def7/6282503b-e4ab-454b-a074-f701a067f39b/cecfe08a-2de2-4171-9051-c68b429ab9e8"
-					(reference "#PWR044")
-					(unit 1)
-				)
+					(reference "#PWR061")
+					(unit 1)
+				)
