File: Buttond_LEDs_IO.kicad_sch (KiCad schematic)
At the start: 14 parts, among them J13 SFH11-PBPC-D05-ST-BK, SW1 RESET, SW2 BOOT

Commit message: ravi's bs
Parts:
- R24, R25, R26, R27: value 1k -> 120
Connections:
- net GND: now also J13.1 (GND), J13.2 (GND); no longer J13.10 (GND), J13.9 (GND)
- net IO10: now also J13.10 (CH0); no longer J13.1 (CH0)
- net IO12: now also J13.9 (CH1); no longer J13.2 (CH1)
- net IO4: now also J13.4 (CH6); no longer J13.7 (CH6)
- net IO5: now also J13.3 (CH7); no longer J13.8 (CH7)
- net IO6: now also J13.6 (CH4); no longer J13.5 (CH4)
- net IO7: now also J13.5 (CH5); no longer J13.6 (CH5)
- net IO8: now also J13.8 (CH2); no longer J13.3 (CH2)
- net IO9: now also J13.7 (CH3); no longer J13.4 (CH3)
Changed lines of the file:
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@@
 	)
 	(junction
-		(at 236.855 104.775)
+		(at 236.855 106.045)
 		(diameter 0)
 		(color 0 0 0 0)
@@
 	(wire
 		(pts
-			(xy 238.125 89.535) (xy 241.935 89.535)
+			(xy 238.125 88.265) (xy 241.935 88.265)
 		)
 		(stroke
@@
 	(wire
 		(pts
-			(xy 238.125 92.075) (xy 241.935 92.075)
+			(xy 238.125 90.805) (xy 241.935 90.805)
 		)
 		(stroke
@@
 	(wire
 		(pts
-			(xy 238.125 94.615) (xy 241.935 94.615)
+			(xy 238.125 93.345) (xy 241.935 93.345)
 		)
 		(stroke
@@
 	(wire
 		(pts
-			(xy 238.125 84.455) (xy 241.935 84.455)
+			(xy 238.125 83.185) (xy 241.935 83.185)
 		)
 		(stroke
@@
 	(wire
 		(pts
-			(xy 236.855 102.235) (xy 236.855 104.775)
+			(xy 236.855 103.505) (xy 236.855 106.045)
 		)
 		(stroke
@@
 	(wire
 		(pts
-			(xy 238.125 99.695) (xy 241.935 99.695)
+			(xy 238.125 98.425) (xy 241.935 98.425)
 		)
 		(stroke
@@
 	(wire
 		(pts
-			(xy 236.855 104.775) (xy 241.935 104.775)
-		)
-		(stroke
-			(width 0)
-			(type default)
-		)
-	)
-	(wire
-		(pts
-			(xy 238.125 81.915) (xy 241.935 81.915)
+			(xy 236.855 106.045) (xy 241.935 106.045)
+		)
+		(stroke
+			(width 0)
+			(type default)
+		)
+	)
+	(wire
+		(pts
+			(xy 238.125 80.645) (xy 241.935 80.645)
 		)
 		(stroke
@@
 	(wire
 		(pts
-			(xy 238.125 97.155) (xy 241.935 97.155)
-		)
-		(stroke
-			(width 0)
-			(type default)
-		)
-	)
-	(wire
-		(pts
-			(xy 238.125 86.995) (xy 241.935 86.995)
+			(xy 238.125 95.885) (xy 241.935 95.885)
+		)
+		(stroke
+			(width 0)
+			(type default)
+		)
+	)
+	(wire
+		(pts
+			(xy 238.125 85.725) (xy 241.935 85.725)
 		)
 		(stroke
@@
 	(wire
 		(pts
-			(xy 241.935 102.235) (xy 236.855 102.235)
+			(xy 241.935 103.505) (xy 236.855 103.505)
 		)
 		(stroke
@@
 	(hierarchical_label "IO9"
 		(shape input)
-		(at 238.125 89.535 180)
+		(at 238.125 88.265 180)
 		(effects
 			(font
@@
 	(hierarchical_label "IO5"
 		(shape input)
-		(at 238.125 99.695 180)
+		(at 238.125 98.425 180)
 		(effects
 			(font
@@
 	(hierarchical_label "IO4"
 		(shape input)
-		(at 238.125 97.155 180)
+		(at 238.125 95.885 180)
 		(effects
 			(font
@@
 	(hierarchical_label "IO10"
 		(shape input)
-		(at 238.125 81.915 180)
+		(at 238.125 80.645 180)
 		(effects
 			(font
@@
 	(hierarchical_label "IO6"
 		(shape input)
-		(at 238.125 92.075 180)
+		(at 238.125 90.805 180)
 		(effects
 			(font
@@
 	(hierarchical_label "IO7"
 		(shape input)
-		(at 238.125 94.615 180)
+		(at 238.125 93.345 180)
 		(effects
 			(font
@@
 	(hierarchical_label "IO12"
 		(shape input)
-		(at 238.125 84.455 180)
+		(at 238.125 83.185 180)
 		(effects
 			(font
@@
 	(hierarchical_label "IO8"
 		(shape input)
-		(at 238.125 86.995 180)
+		(at 238.125 85.725 180)
 		(effects
 			(font
@@
 		(fields_autoplaced yes)
 		(property "Reference" "R24"
-			(at 131.445 82.5499 0)
+			(at 130.81 82.5499 0)
 			(effects
 				(font
@@
 			)
 		)
-		(property "Value" "1k"
-			(at 131.445 85.0899 0)
+		(property "Value" "120"
+			(at 130.81 85.0899 0)
 			(effects
 				(font
@@
 	(symbol
 		(lib_id "power:GND")
-		(at 236.855 104.775 0)
+		(at 236.855 106.045 0)
 		(unit 1)
 		(exclude_from_sim no)
@@
 		(fields_autoplaced yes)
 		(property "Reference" "#PWR067"
+			(at 236.855 112.395 0)
+			(effects
+				(font
+					(size 1.27 1.27)
+				)
+				(hide yes)
+			)
+		)
+		(property "Value" "GND"
 			(at 236.855 111.125 0)
 			(effects
@@
 					(size 1.27 1.27)
 				)
-				(hide yes)
-			)
-		)
-		(property "Value" "GND"
-			(at 236.855 109.855 0)
-			(effects
-				(font
-					(size 1.27 1.27)
-				)
 			)
 		)
 		(property "Footprint" ""
-			(at 236.855 104.775 0)
+			(at 236.855 106.045 0)
 			(effects
 				(font
@@
 		)
 		(property "Datasheet" ""
-			(at 236.855 104.775 0)
+			(at 236.855 106.045 0)
 			(effects
 				(font
@@
 		)
 		(property "Description" "Power symbol creates a global label with name \"GND\" , ground"
-			(at 236.855 104.775 0)
+			(at 236.855 106.045 0)
 			(effects
 				(font
@@
 		(fields_autoplaced yes)
 		(property "Reference" "R25"
-			(at 142.875 82.5499 0)
+			(at 142.24 82.5499 0)
 			(effects
 				(font
@@
 			)
 		)
-		(property "Value" "1k"
-			(at 142.875 85.0899 0)
+		(property "Value" "120"
+			(at 142.24 85.0899 0)
 			(effects
 				(font
@@
 		(fields_autoplaced yes)
 		(property "Reference" "R26"
-			(at 154.305 82.5499 0)
+			(at 153.67 82.5499 0)
 			(effects
 				(font
@@
 			)
 		)
-		(property "Value" "1k"
-			(at 154.305 85.0899 0)
+		(property "Value" "120"
+			(at 153.67 85.0899 0)
 			(effects
 				(font
@@
 		(fields_autoplaced yes)
 		(property "Reference" "R27"
-			(at 165.735 82.5499 0)
+			(at 165.1 82.5499 0)
 			(effects
 				(font
@@
 			)
 		)
-		(property "Value" "1k"
-			(at 165.735 85.0899 0)
-			(effects
-				(font
+		(property "Value" "120"
+			(at 165.1 85.0899 0)
+			(effects
+				(font

Commit message: start of RevB. BOM for revA
Parts:
- C18: Mouser Part Number (none) -> 963-HMK107B7104KA-T; P/N (none) -> HMK107B7104KA-T
- LV1, LV2, LV3, LV4: P/N (none) -> XL-1608UBC-06A
- R22, R23: Mouser Part Number (none) -> 71-CRCW060310K0FKEI; P/N (none) -> CRCW060310K0FKEI
- R24, R25, R26, R27: Mouser Part Number (none) -> 71-CRCW0603120RFKEC; P/N (none) -> CRCW0603120RFKEC
- SW1: Mouser Part Number (none) -> 667-EVQ-7Q203W; P/N (none) -> EVQ-7Q203W
- SW2: Mouser Part Number (none) -> 229-CJS-1200TA; P/N (none) -> CJS-1200TA
Changed lines of the file:
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@@
+			)
+		)
+		(property "P/N" "CJS-1200TA"
+			(at 71.12 105.41 0)
+			(effects
+				(font
+					(size 1.27 1.27)
+				)
+			)
+		)
+		(property "Mouser Part Number" "229-CJS-1200TA"
+			(at 71.12 105.41 0)
+			(effects
+				(font
+					(size 1.27 1.27)
+				)
 			)
 		)
@@
 			)
 		)
+		(property "P/N" "XL-1608UBC-06A"
+			(at 128.905 92.71 0)
+			(effects
+				(font
+					(size 1.27 1.27)
+				)
+			)
+		)
 		(pin "1"
 		)
@@
 				)
 				(hide yes)
+			)
+		)
+		(property "P/N" "CRCW0603120RFKEC"
+			(at 128.905 83.82 0)
+			(effects
+				(font
+					(size 1.27 1.27)
+				)
+			)
+		)
+		(property "Mouser Part Number" " 71-CRCW0603120RFKEC"
+			(at 128.905 83.82 0)
+			(effects
+				(font
+					(size 1.27 1.27)
+				)
 			)
 		)
@@
 			)
 		)
+		(property "P/N" "HMK107B7104KA-T"
+			(at 60.96 68.58 0)
+			(effects
+				(font
+					(size 1.27 1.27)
+				)
+			)
+		)
+		(property "Mouser Part Number" "963-HMK107B7104KA-T"
+			(at 60.96 68.58 0)
+			(effects
+				(font
+					(size 1.27 1.27)
+				)
+			)
+		)
 		(pin "1"
 		)
@@
 			)
 		)
+		(property "P/N" "CRCW060310K0FKEI"
+			(at 60.96 55.88 0)
+			(effects
+				(font
+					(size 1.27 1.27)
+				)
+			)
+		)
+		(property "Mouser Part Number" "71-CRCW060310K0FKEI"
+			(at 60.96 55.88 0)
+			(effects
+				(font
+					(size 1.27 1.27)
+				)
+			)
+		)
 		(pin "1"
 		)
@@
 			)
 		)
+		(property "P/N" "CRCW0603120RFKEC"
+			(at 140.335 83.82 0)
+			(effects
+				(font
+					(size 1.27 1.27)
+				)
+			)
+		)
+		(property "Mouser Part Number" " 71-CRCW0603120RFKEC"
+			(at 140.335 83.82 0)
+			(effects
+				(font
+					(size 1.27 1.27)
+				)
+			)
+		)
 		(pin "1"
 		)
@@
 				)
 				(hide yes)
+			)
+		)
+		(property "P/N" "XL-1608UBC-06A"
+			(at 140.335 92.71 0)
+			(effects
+				(font
+					(size 1.27 1.27)
+				)
 			)
 		)
@@
 			)
 		)
+		(property "P/N" "CRCW0603120RFKEC"
+			(at 151.765 83.82 0)
+			(effects
+				(font
+					(size 1.27 1.27)
+				)
+			)
+		)
+		(property "Mouser Part Number" " 71-CRCW0603120RFKEC"
+			(at 151.765 83.82 0)
+			(effects
+				(font
+					(size 1.27 1.27)
+				)
+			)
+		)
 		(pin "1"
 		)
@@
 				)
 				(hide yes)
+			)
+		)
+		(property "P/N" "CRCW0603120RFKEC"
+			(at 163.195 83.82 0)
+			(effects
+				(font
+					(size 1.27 1.27)
+				)
+			)
+		)
+		(property "Mouser Part Number" " 71-CRCW0603120RFKEC"
+			(at 163.195 83.82 0)
+			(effects
+				(font
+					(size 1.27 1.27)
+				)
 			)
 		)
@@
 			)
 		)
+		(property "P/N" "EVQ-7Q203W"
+			(at 71.12 63.5 0)
+			(effects
+				(font
+					(size 1.27 1.27)
+				)
+			)
+		)
+		(property "Mouser Part Number" "667-EVQ-7Q203W"
+			(at 71.12 63.5 0)
+			(effects
+				(font
+					(size 1.27 1.27)
+				)
+			)
+		)
 		(pin "2"
 		)
@@
 				)
 				(hide yes)
+			)
+		)
+		(property "P/N" "XL-1608UBC-06A"
+			(at 163.195 92.71 0)
+			(effects
+				(font
+					(size 1.27 1.27)
+				)
 			)
 		)
@@
 			)
 		)
+		(property "P/N" "XL-1608UBC-06A"
+			(at 151.765 92.71 0)
+			(effects
+				(font
+					(size 1.27 1.27)
+				)
+			)
+		)
 		(pin "1"
 		)
@@
 			)
 		)
+		(property "P/N" "CRCW060310K0FKEI"
+			(at 60.325 105.41 0)
+			(effects
+				(font
+					(size 1.27 1.27)
+				)
+			)
+		)
+		(property "Mouser Part Number" "71-CRCW060310K0FKEI"
+			(at 60.325 105.41 0)
+			(effects
+				(font
+					(size 1.27 1.27)
+				)
+			)
+		)

Commit message: workday
Parts:
- C18: footprint Capacitor_SMD:C_0603_1608Metric -> Capacitor_SMD:C_0603_1608Metric_Pad1.08x0.95mm_HandSolder
- R22, R23, R24, R25, R26, R27: footprint Resistor_SMD:R_0603_1608Metric -> Resistor_SMD:R_0603_1608Metric_Pad0.98x0.95mm_HandSolder
Changed lines of the file:
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@@
 			)
 		)
-		(property "Footprint" "Resistor_SMD:R_0603_1608Metric"
+		(property "Footprint" "Resistor_SMD:R_0603_1608Metric_Pad0.98x0.95mm_HandSolder"
 			(at 129.921 84.074 90)
 			(effects
@@
 			)
 		)
-		(property "Footprint" "Capacitor_SMD:C_0603_1608Metric"
+		(property "Footprint" "Capacitor_SMD:C_0603_1608Metric_Pad1.08x0.95mm_HandSolder"
 			(at 59.9948 72.39 0)
 			(effects
@@
 			)
 		)
-		(property "Footprint" "Resistor_SMD:R_0603_1608Metric"
+		(property "Footprint" "Resistor_SMD:R_0603_1608Metric_Pad0.98x0.95mm_HandSolder"
 			(at 59.944 56.134 90)
 			(effects
@@
 			)
 		)
-		(property "Footprint" "Resistor_SMD:R_0603_1608Metric"
+		(property "Footprint" "Resistor_SMD:R_0603_1608Metric_Pad0.98x0.95mm_HandSolder"
 			(at 141.351 84.074 90)
 			(effects
@@
 			)
 		)
-		(property "Footprint" "Resistor_SMD:R_0603_1608Metric"
+		(property "Footprint" "Resistor_SMD:R_0603_1608Metric_Pad0.98x0.95mm_HandSolder"
 			(at 152.781 84.074 90)
 			(effects
@@
 			)
 		)
-		(property "Footprint" "Resistor_SMD:R_0603_1608Metric"
+		(property "Footprint" "Resistor_SMD:R_0603_1608Metric_Pad0.98x0.95mm_HandSolder"
 			(at 164.211 84.074 90)
 			(effects
@@
 			)
 		)
-		(property "Footprint" "Resistor_SMD:R_0603_1608Metric"
+		(property "Footprint" "Resistor_SMD:R_0603_1608Metric_Pad0.98x0.95mm_HandSolder"
 			(at 60.579 106.426 90)
 			(effects

Commit message: rev B
Parts:
- LV1, LV2, LV3, LV4: footprint LED_SMD:LED_0603_1608Metric -> LED_SMD:LED_0603_1608Metric_Pad1.05x0.95mm_HandSolder
- SW1: footprint UTSVT_Special:SW_SPST_B3SL-1002P -> Boot Switch:TL3365AF180QG
Connections:
- net IO10: now also J13.4 (CH6); no longer J13.10 (CH0)
- net IO12: now also J13.3 (CH7); no longer J13.9 (CH1)
- net IO4: now also J13.10 (CH0); no longer J13.4 (CH6)
- net IO5: now also J13.9 (CH1); no longer J13.3 (CH7)
- net IO6: now also J13.8 (CH2); no longer J13.6 (CH4)
- net IO7: now also J13.7 (CH3); no longer J13.5 (CH5)
- net IO8: now also J13.6 (CH4); no longer J13.8 (CH2)
- net IO9: now also J13.5 (CH5); no longer J13.7 (CH3)
Changed lines of the file:
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@@
 		)
 	)
-	(hierarchical_label "IO9"
+	(hierarchical_label "IO5"
 		(shape input)
-		(at 238.125 88.265 180)
+		(at 238.125 83.185 180)
 		(effects
 			(font
@@
 		)
 	)
+	(hierarchical_label "IO10"
+		(shape input)
+		(at 238.125 95.885 180)
+		(effects
+			(font
+				(size 1.27 1.27)
+			)
+			(justify right)
+		)
+	)
+	(hierarchical_label "IO9"
+		(shape input)
+		(at 238.125 93.345 180)
+		(effects
+			(font
+				(size 1.27 1.27)
+			)
+			(justify right)
+		)
+	)
 	(hierarchical_label "Reset"
 		(shape output)
@@
 		)
 	)
-	(hierarchical_label "IO5"
+	(hierarchical_label "IO7"
 		(shape input)
-		(at 238.125 98.425 180)
-		(effects
-			(font
-				(size 1.27 1.27)
-			)
-			(justify right)
-		)
-	)
-	(hierarchical_label "IO4"
-		(shape input)
-		(at 238.125 95.885 180)
+		(at 238.125 88.265 180)
 		(effects
 			(font
@@
 		)
 	)
-	(hierarchical_label "IO10"
-		(shape input)
-		(at 238.125 80.645 180)
-		(effects
-			(font
-				(size 1.27 1.27)
-			)
-			(justify right)
-		)
-	)
 	(hierarchical_label "LED1"
 		(shape input)
@@
 	(hierarchical_label "IO6"
 		(shape input)
-		(at 238.125 90.805 180)
+		(at 238.125 85.725 180)
 		(effects
 			(font
@@
 		)
 	)
-	(hierarchical_label "IO7"
+	(hierarchical_label "IO4"
 		(shape input)
-		(at 238.125 93.345 180)
+		(at 238.125 80.645 180)
+		(effects
+			(font
+				(size 1.27 1.27)
+			)
+			(justify right)
+		)
+	)
+	(hierarchical_label "IO12"
+		(shape input)
+		(at 238.125 98.425 180)
 		(effects
 			(font
@@
 		)
 	)
-	(hierarchical_label "IO12"
+	(hierarchical_label "IO8"
 		(shape input)
-		(at 238.125 83.185 180)
+		(at 238.125 90.805 180)
 		(effects
 			(font
@@
 		)
 	)
-	(hierarchical_label "IO8"
-		(shape input)
-		(at 238.125 85.725 180)
-		(effects
-			(font
-				(size 1.27 1.27)
-			)
-			(justify right)
-		)
-	)
 	(symbol
 		(lib_id "Switch:SW_SPDT")
@@
 			)
 		)
-		(property "Footprint" "LED_SMD:LED_0603_1608Metric"
+		(property "Footprint" "LED_SMD:LED_0603_1608Metric_Pad1.05x0.95mm_HandSolder"
 			(at 128.905 92.71 0)
 			(effects
@@
 			)
 		)
-		(property "Footprint" "LED_SMD:LED_0603_1608Metric"
+		(property "Footprint" "LED_SMD:LED_0603_1608Metric_Pad1.05x0.95mm_HandSolder"
 			(at 140.335 92.71 0)
 			(effects
@@
 			)
 		)
-		(property "Footprint" "UTSVT_Special:SW_SPST_B3SL-1002P"
+		(property "Footprint" "Boot Switch:TL3365AF180QG"
 			(at 71.12 58.42 0)
 			(effects
@@
 			)
 		)
-		(property "Footprint" "LED_SMD:LED_0603_1608Metric"
+		(property "Footprint" "LED_SMD:LED_0603_1608Metric_Pad1.05x0.95mm_HandSolder"
 			(at 163.195 92.71 0)
 			(effects
@@
 			)
 		)
-		(property "Footprint" "LED_SMD:LED_0603_1608Metric"
+		(property "Footprint" "LED_SMD:LED_0603_1608Metric_Pad1.05x0.95mm_HandSolder"
 			(at 151.765 92.71 0)
 			(effects
