File: VehicleControlUnit.kicad_pcb (KiCad board)
At the start: 4 copper layers, 95 x 100 mm, 99 parts, among them Con1 LED, Con2 LED, J1 Conn_01x02, J10 CAR_CAN_OUT, J11 CAR_CAN_Breakout, J12 USB_C_Receptacle_USB2.0_16P, J13 UART_Breakout, J14 Conn_01x04, J15 Conn_01x04, J16 IO_Breakout, J2 Precharge_Ready, J4 Precharge+_Conn, J5 Precharge-_Conn, J6 MOTOR_CAN_IN, J7 MOTOR_CAN_OUT, J8 MOTOR_CAN_Breakout, J9 CAR_CAN_IN, Q1 Q_PMOS_GDS, Q2 IRLML0030, Q3 IRLML0030, SW1 RESET, SW2 BOOT, U1 TLV1117LV33DCYR, U3 ESP32-C6-MINI-1/U, U4 TCMT1106, U5 TCMT1106

Commit message: first revision
Parts:
- added J17: IO_5-8, Connector_PinHeader_2.54mm:PinHeader_1x04_P2.54mm_Vertical, F.Cu at (123.4, 128.0)
- added J18: IO_9-12, Connector_PinHeader_2.54mm:PinHeader_1x04_P2.54mm_Vertical, F.Cu at (123.4, 105.9)
- D7: renamed from D6; moved to F.Cu
- D8: renamed from D7; moved to F.Cu
- J12: footprint Connector_USB:USB_C_Receptacle_GCT_USB4105-xx-A_16P_TopMnt_Horizontal -> USBC:GCT_USB4215-03-A_REVA
- J16: value IO_Breakout -> IO_1-4
- R13, R14: moved to B.Cu
- moved J12 112.1 mm to (134.2, 138.2), turned to 0 degrees
- moved R13 110.6 mm to (127.0, 136.3), turned to 180 degrees
- moved J1 105.6 mm to (150.2, 138.1), turned to 0 degrees
- moved D6 104.9 mm to (131.8, 131.3), turned to 0 degrees
- moved C5 102.1 mm to (122.0, 120.1), turned to 90 degrees
- moved D4 100.0 mm to (135.7, 131.3), turned to 180 degrees
- moved U2 99.1 mm to (124.1, 120.3), turned to 180 degrees
- moved LV1 98.3 mm to (148.3, 132.2), turned to 90 degrees
- moved R11 98.2 mm to (125.6, 117.3), turned to 0 degrees
- moved R12 98.1 mm to (124.1, 123.3), turned to 180 degrees
- moved R14 98.0 mm to (141.5, 136.3), turned to 0 degrees
- moved R4 96.3 mm to (149.3, 131.2), turned to 180 degrees
- moved C3 95.5 mm to (127.0, 119.3), turned to 0 degrees
- moved C11 94.8 mm to (139.0, 130.5), turned to 90 degrees
- moved C9 94.8 mm to (127.0, 121.3), turned to 0 degrees
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- renumbered C10 to C11, C11 to C12, C12 to C13, C13 to C14, C14 to C15, C15 to C16, C16 to C17, D9 to D10, D5 to D6, D8 to D9
Connections:
- J3 pad 18: /VPrecharge+ -> /ISO_ADC_CLK
- J3 pad 20: /ISO_ADC_CLK -> /VPrecharge+
- U3 pad 10: unconnected-(U3-MTDI/GPIO5/ADC1_CH5-Pad10) -> /ESP/IO12
- U3 pad 12: unconnected-(U3-GPIO0/ADC1_CH0/XTAL_32K_P-Pad12) -> /ESP/IO5
- U3 pad 13: unconnected-(U3-GPIO1/ADC1_CH1/XTAL_32K_N-Pad13) -> /ESP/IO6
- U3 pad 15: unconnected-(U3-MTCK/GPIO6/ADC1_CH6-Pad15) -> /ESP/IO7
- U3 pad 16: unconnected-(U3-MTDO/GPIO7-Pad16) -> /ESP/IO8
- U3 pad 5: unconnected-(U3-GPIO2/ADC1_CH2-Pad5) -> /ESP/IO9
- U3 pad 6: unconnected-(U3-GPIO3/ADC1_CH3-Pad6) -> /ESP/IO10
- U3 pad 9: unconnected-(U3-MTMS/GPIO4/ADC1_CH4-Pad9) -> /ESP/IO11
Routing:
- net /3V3_LSOM: track 0.00 -> 133.8 mm, vias 0 -> 6
- net /C_CAN_H: track 0.00 -> 75.2 mm, vias 0 -> 2
- net /C_CAN_L: track 0.00 -> 74.1 mm, vias 0 -> 2
- net /ISO_ADC_CLK: track 0.00 -> 71.4 mm, vias 0 -> 1
- net /VPrecharge-: track 0.00 -> 70.2 mm, vias 0 -> 1
- net /M_CAN_H: track 0.00 -> 69.3 mm
- net /M_CAN_L: track 0.00 -> 68.0 mm, vias 0 -> 2
- net /M_Sense: track 0.00 -> 67.5 mm, vias 0 -> 3
- net /ESP/RESET: track 0.00 -> 56.0 mm, vias 0 -> 3
- net /VPrecharge+: track 0.00 -> 53.5 mm, vias 0 -> 1
- net /Precharge_Ready: track 0.00 -> 50.5 mm, vias 0 -> 2
- net /MPre_Sense: track 0.00 -> 46.8 mm, vias 0 -> 2
- net /ESP_RX: track 0.00 -> 45.7 mm, vias 0 -> 1
- net /ESP_TX: track 0.00 -> 42.9 mm, vias 0 -> 2
- net /M_Enable: track 0.00 -> 39.2 mm, vias 0 -> 1
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- added copper zone on B.Cu, net GND
- added copper zone on F.Cu, net GND
Other:
- board size 95 x 100 mm -> 86.6 x 100.1 mm
- board text added: "CAN_BREAKOUT"
- board text added: "UART_BREAKOUT"

Commit message: tweaking
Parts:
- added G***: LOGO, UTSVT_Special:Hallock_Image, F.Cu at (179.3, 59.1)
- added G***: LOGO, LOGO, F.Cu at (154.0, 56.0)
- added G***: LOGO, LOGO, F.Cu at (159.0, 67.0)
- added G***: LOGO, UTSVT_Special:UTSVT_Logo_Symbol, F.Cu at (179.6, 130.8)
- added G***: LOGO, LOGO, B.Cu at (134.1, 98.0)
- R17, R22: value 1k -> 2k
- moved M_Pre_Sen_TP1 48.4 mm to (180.6, 98.6)
- moved M_Sen_TP1 3.36 mm to (180.5, 93.4)
- moved C1 1.99 mm to (119.2, 102.9), turned to -90 degrees
- moved D6 1.33 mm to (131.0, 132.3)
- moved C8 1.12 mm to (126.8, 112.7)
- moved C3 1.12 mm to (125.9, 119.3)
- moved C5 1.12 mm to (120.9, 120.0)
- moved C6 1.12 mm to (129.7, 112.7)
- moved C9 1.12 mm to (125.9, 121.3)
- moved J13 1.12 mm to (145.9, 94.6)
- moved J16 1.12 mm to (146.0, 108.6)
- moved J17 1.12 mm to (122.3, 128.0)
- moved J18 1.12 mm to (122.3, 105.9)
- moved LV6 1.12 mm to (149.4, 118.9)
- moved LV7 1.12 mm to (149.4, 116.7)
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Routing:
- net /MPre_Sense: track 46.8 -> 68.4 mm, vias 2 -> 3
- net /ESP/VBUSB: track 8.07 -> 9.78 mm
- net /M_Sense: track 67.5 -> 65.8 mm
- net /VPrecharge+: track 53.5 -> 55.1 mm
- net /3V3_LSOM: track 133.8 -> 132.6 mm
- net /ESP/BOOT: track 37.5 -> 38.6 mm
- net /ESP_RX: track 45.7 -> 46.9 mm
- net /ESP/RESET: track 56.0 -> 57.2 mm
- net /ESP/3V3_USB: track 33.5 -> 34.6 mm
- net /ESP_TX: track 42.9 -> 43.9 mm
- net /ESP/USB_D-: track 16.2 -> 17.1 mm
- net /ISO_ADC_CLK: track 71.4 -> 72.0 mm
- net /Precharge_Ready: track 50.5 -> 50.0 mm
- net GND: vias 78 -> 128
- added copper zone on In2.Cu, net GND
Other:
- board size 86.6 x 100.1 mm -> 86.6 x 100 mm

Commit message: fixed
Parts:
- removed C17: 0.1u, Capacitor_SMD:C_0805_2012Metric
- removed D10: D, Active-PrechargeLib:SODFL4724X108N
- removed the G*** at (179.3, 59.1)
- removed the G*** at (179.6, 130.8)
- removed J18: IO_9-12, Connector_PinHeader_2.54mm:PinHeader_1x04_P2.54mm_Vertical
- added C10: 10u, Capacitor_SMD:C_0603_1608Metric, F.Cu at (132.4, 110.2)
- added D5: TVS, Diode_SMD:D_0603_1608Metric, F.Cu at (119.3, 117.8)
- C1, C15, C16, C2, C3, C4, C5, C6, C7, C8, C9, D4, D6, D9, Q1, R1, R10, R11, R12, R13, R14, R15, R16, R17, R18, R19, R2, R20, R21, R22, R23, R24, R25, R26, R27, R28, R29, R3, R30, R4, R5, R6, R7, R8, R9: moved to F.Cu
- C11: value 10u -> 1u; footprint Capacitor_SMD:C_0603_1608Metric -> Capacitor_SMD:C_0805_2012Metric; moved to F.Cu
- C12, C14: value 1u -> 0.1u; moved to F.Cu
- C13: value 0.1u -> 1u; moved to F.Cu
- D8: value TVS -> D; footprint Diode_SMD:D_0603_1608Metric -> Active-PrechargeLib:SODFL4724X108N
- J10, J2, J4, J5, J9: footprint utsvt_conn:Molex_MicroFit3.0_1x2xP3.00mm_PolarizingPeg_Vertical -> Connector_Molex:Molex_Nano-Fit_105309-xx02_1x02_P2.50mm_Vertical
- J16: value IO_1-4 -> Conn_01x04
- J17: value IO_5-8 -> Conn_01x08; footprint Connector_PinHeader_2.54mm:PinHeader_1x04_P2.54mm_Vertical -> Connector_PinHeader_2.54mm:PinHeader_1x08_P2.54mm_Vertical
- J6, J7: footprint utsvt_conn:Molex_MicroFit3.0_1x4xP3.00mm_PolarizingPeg_Vertical -> Connector_Molex:Molex_Nano-Fit_105309-xx04_1x04_P2.50mm_Vertical
- moved J4 77.4 mm to (189.6, 127.7), turned to 180 degrees
- moved J5 75.7 mm to (189.5, 118.7), turned to 180 degrees
- moved D8 69.8 mm to (125.5, 56.9)
- moved C11 62.5 mm to (133.3, 68.2), turned to 180 degrees
- moved C15 61.6 mm to (178.1, 104.4), turned to 90 degrees
- moved M_Pre_Sen_TP1 53.5 mm to (127.2, 94.2)
- moved R14 28.6 mm to (113.9, 130.0), turned to -90 degrees
- moved C13 28.0 mm to (133.3, 88.3), turned to 180 degrees
- moved J16 27.8 mm to (118.3, 105.8), turned to 90 degrees
- moved J12 27.7 mm to (112.0, 122.8), turned to -90 degrees
- moved D2 26.5 mm to (125.0, 113.1), turned to 0 degrees
- moved U3 26.1 mm to (125.6, 138.1), turned to 180 degrees
- moved C8 26.0 mm to (136.6, 136.8)
- moved LV6 25.5 mm to (147.3, 93.4), turned to -90 degrees
- moved R13 25.5 mm to (113.9, 115.6), turned to 90 degrees
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Connections:
- C11 pad 1: /ESP/5V_USB -> GND
- C11 pad 2: GND -> /M_Sense
- C12 pad 1: GND -> Net-(J14-Pin_2)
- C12 pad 2: /M_Sense -> GND
- C13 pad 1: Net-(J14-Pin_2) -> GND
- C13 pad 2: GND -> /MPre_Sense
- C14 pad 1: GND -> Net-(J15-Pin_2)
- C14 pad 2: /MPre_Sense -> GND
- C15 pad 1: Net-(J15-Pin_2) -> /ESP/RESET
- C16 pad 1: /ESP/RESET -> /ESP/BOOT
- D6 pad 2: /ESP/VBUSB -> /ESP/USB_D-
- D7 pad 2: /ESP/USB_D- -> /ESP/USB_D+
- D8 pad 1: GND -> /LV+
- D8 pad 2: /ESP/USB_D+ -> /ContactorDriver/MCon-
- D9 pad 2: /ContactorDriver/MCon- -> /ContactorDriver/M_PreCon-
- U3 pad 10: /ESP/IO12 -> /ESP/IO9
- U3 pad 12: /ESP/IO5 -> /ESP/IO8
- U3 pad 13: /ESP/IO6 -> /ESP/IO7
- U3 pad 15: /ESP/IO7 -> /ESP/IO6
- U3 pad 16: /ESP/IO8 -> /ESP/IO5
- U3 pad 26: /ESP/IO1 -> /ESP/IO4
- U3 pad 27: /ESP/IO2 -> /ESP/IO3
- U3 pad 28: /ESP/IO3 -> /ESP/IO2
- U3 pad 29: /ESP/IO4 -> /ESP/IO1
- U3 pad 5: /ESP/IO9 -> /ESP/IO12
- U3 pad 6: /ESP/IO10 -> /ESP/IO11
- U3 pad 9: /ESP/IO11 -> /ESP/IO10
Routing:
- net /3V3_LSOM: track 132.6 -> 40.8 mm
- net /ESP/LED1: track 13.3 -> 46.2 mm, vias 1 -> 2
- net /ESP/LED4: track 10.9 -> 43.6 mm, vias 1 -> 2
- net /ESP_TX: track 43.9 -> 75.7 mm, vias 2 -> 3
- net /ESP/LED3: track 10.5 -> 41.8 mm, vias 1 -> 2
- net /ESP_RX: track 46.9 -> 75.3 mm, vias 1 -> 2
- net /ESP/LED2: track 13.2 -> 41.4 mm, vias 1 -> 2
- net /MPre_Sense: track 68.4 -> 46.1 mm, vias 3 -> 2
- net /ESP/IO1: track 13.3 -> 34.5 mm, vias 0 -> 1
- net /LV+: track 2.00 -> 21.1 mm, vias 13 -> 7
- net /ESP/3V3: track 19.9 -> 38.9 mm, vias 4 -> 2
- net /ESP/BOOT: track 38.6 -> 56.4 mm, vias 1 -> 3
- net /M_CAN_L: track 68.0 -> 52.0 mm, vias 2 -> 0
- net /ESP/IO2: track 15.6 -> 31.6 mm, vias 0 -> 1
- net /VPrecharge-: track 70.2 -> 54.3 mm
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- added copper zone on B.Cu, net /3V3_LSOM
Other:
- board text added: "CAN_H"
- board text added: "CAN_L"
- board text added: "ESP LEDS"
- board text added: "LSOM LEDS"

Commit message: review changes
Parts:
- removed J17: Conn_01x08, Connector_PinHeader_2.54mm:PinHeader_1x08_P2.54mm_Vertical
- added G***: LOGO, UTSVT_Special:UTSVT_Logo_Symbol, F.Cu at (149.3, 121.0)
- added G***: LOGO, LOGO, B.Cu at (184.5, 70.0)
- added G***: LOGO, LOGO, B.Cu at (174.2, 58.1)
- G***: moved to F.Cu
- J10: value CAR_CAN_OUT -> CAR_CAN_Breakout; footprint Connector_Molex:Molex_Nano-Fit_105309-xx02_1x02_P2.50mm_Vertical -> Connector_PinHeader_2.54mm:PinHeader_1x02_P2.54mm_Vertical
- J11: value CAR_CAN_Breakout -> USB_C_Receptacle_USB2.0_16P; footprint Connector_PinHeader_2.54mm:PinHeader_1x02_P2.54mm_Vertical -> USBC:GCT_USB4215-03-A_REVA
- J12: value USB_C_Receptacle_USB2.0_16P -> UART_Breakout; footprint USBC:GCT_USB4215-03-A_REVA -> Connector_PinHeader_2.54mm:PinHeader_1x02_P2.54mm_Vertical
- J13: value UART_Breakout -> Conn_01x04; footprint Connector_PinHeader_2.54mm:PinHeader_1x02_P2.54mm_Vertical -> utsvt_conn:Molex_MicroFit3.0_1x4xP3.00mm_PolarizingPeg_Vertical
- J15: footprint utsvt_conn:Molex_MicroFit3.0_1x4xP3.00mm_PolarizingPeg_Vertical -> Connector_PinHeader_2.54mm:PinHeader_1x04_P2.54mm_Vertical
- J16: value Conn_01x04 -> Conn_01x08; footprint Connector_PinHeader_2.54mm:PinHeader_1x04_P2.54mm_Vertical -> Connector_PinHeader_2.54mm:PinHeader_1x08_P2.54mm_Vertical
- J6: value MOTOR_CAN_IN -> Conn_02x04_Counter_Clockwise; footprint Connector_Molex:Molex_Nano-Fit_105309-xx04_1x04_P2.50mm_Vertical -> utsvt_conn:Molex_MicroFit3.0_2x4xP3.00mm_PolarizingPeg_Vertical
- J7: value MOTOR_CAN_OUT -> MOTOR_CAN_Breakout; footprint Connector_Molex:Molex_Nano-Fit_105309-xx04_1x04_P2.50mm_Vertical -> Connector_PinHeader_2.54mm:PinHeader_1x02_P2.54mm_Vertical
- J8: value MOTOR_CAN_Breakout -> CAR_CAN_IN; footprint Connector_PinHeader_2.54mm:PinHeader_1x02_P2.54mm_Vertical -> Connector_Molex:Molex_Nano-Fit_105309-xx02_1x02_P2.50mm_Vertical
- J9: value CAR_CAN_IN -> CAR_CAN_OUT
- moved J11 56.4 mm to (112.0, 122.8), turned to -90 degrees
- moved J12 53.7 mm to (155.1, 90.8), turned to 0 degrees
- moved J13 53.2 mm to (114.0, 56.9), turned to -90 degrees
- moved J8 43.6 mm to (178.2, 135.8), turned to 90 degrees
- moved J15 29.2 mm to (118.3, 105.8), turned to 90 degrees
- moved J16 26.8 mm to (141.3, 119.5), turned to 0 degrees
- moved J7 22.1 mm to (167.9, 93.3)
- moved J14 20.0 mm to (114.0, 76.9)
- moved J10 14.2 mm to (168.4, 125.5)
- moved J6 10.7 mm to (188.6, 99.9), turned to 90 degrees
- moved J4 9.12 mm to (188.5, 118.6)
- moved J5 9.12 mm to (188.4, 109.7)
- moved 12V_TP1 7.20 mm to (156.2, 118.8)
- moved LVGND_TP1 3.06 mm to (176.8, 118.3)
- moved G*** 0.90 mm to (154.8, 55.5)
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Connections:
- net /3V3_LSOM renamed 3V3_LSOM
- 12V_TP1 pad 1: /LV+ -> +12V
- C12 pad 1: Net-(J14-Pin_2) -> Net-(J13-Pin_2)
- C14 pad 1: Net-(J15-Pin_2) -> Net-(J14-Pin_2)
- C2 pad 1: /LV+ -> +12V
- D1 pad 1: /LV+ -> +12V
- D8 pad 1: /LV+ -> +12V
- D9 pad 1: /LV+ -> +12V
- J1 pad 2: +12V -> /LV+
- J13 pad 1: /ESP_TX -> /ContactorDriver/MCon-
- J13 pad 2: /ESP_RX -> Net-(J13-Pin_2)
- J14 pad 1: /ContactorDriver/MCon- -> /ContactorDriver/M_PreCon-
- J14 pad 3: /LV+ -> +12V
- J14 pad 4: /LV+ -> +12V
- J15 pad 1: /ContactorDriver/M_PreCon- -> /ESP/IO1
- J15 pad 2: Net-(J15-Pin_2) -> /ESP/IO2
- J15 pad 3: /LV+ -> /ESP/IO3
- J15 pad 4: /LV+ -> /ESP/IO4
- J16 pad 1: /ESP/IO1 -> /ESP/IO5
- J16 pad 2: /ESP/IO2 -> /ESP/IO6
- J16 pad 3: /ESP/IO3 -> /ESP/IO7
- J16 pad 4: /ESP/IO4 -> /ESP/IO8
- J3 pad 21: /LV+ -> +12V
- J3 pad 22: /LV+ -> +12V
- J3 pad 23: /LV+ -> +12V
- J3 pad 24: /LV+ -> +12V
- J6 pad 1: /LV+ -> +12V
- J7 pad 1: /LV+ -> /M_CAN_H
- J7 pad 2: GND -> /M_CAN_L
- J8 pad 1: /M_CAN_H -> /C_CAN_H
- J8 pad 2: /M_CAN_L -> /C_CAN_L
- Q1 pad 2: /LV+ -> +12V
- Q1 pad 3: +12V -> /LV+
- R17 pad 1: Net-(J14-Pin_2) -> Net-(J13-Pin_2)
- R19 pad 2: /LV+ -> +12V
- R22 pad 1: Net-(J15-Pin_2) -> Net-(J14-Pin_2)
- R24 pad 2: /LV+ -> +12V
- R4 pad 1: /LV+ -> +12V
Routing:
- net +12V: track 4.79 -> 21.5 mm, vias 0 -> 9
- net /M_CAN_H: track 54.0 -> 37.5 mm
- net /LV+: track 21.1 -> 4.79 mm, vias 7 -> 0
- net /M_CAN_L: track 52.0 -> 37.5 mm
- net Net-(J13-Pin_2): track 0.00 -> 12.6 mm
- net Net-(J15-Pin_2): track 12.4 -> 0.00 mm
- net /ISO_ADC_CLK: track 67.1 -> 55.5 mm
- net 3V3_LSOM: track 40.8 -> 31.8 mm
- net /VPrecharge+: track 64.2 -> 55.2 mm
- net /VPrecharge-: track 54.3 -> 45.4 mm
- net /Precharge_Ready: track 47.6 -> 48.8 mm
- net /ESP_TX: track 75.7 -> 76.8 mm
- net /M_Sense: track 58.9 -> 59.9 mm
- net /ContactorDriver/MCon-: track 15.1 -> 16.0 mm
- net /C_CAN_L: track 70.8 -> 71.7 mm
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- added copper zone on In2.Cu, net +12V
- removed copper zone on In2.Cu, net /LV+
Other:
- board text added: "CAN_L CAN_H"
- board text added: "CAR_CAN_BREAKOUT"
- board text added: "MOTOR CAN_BREAKOUT"
- board text added: "TX RX"
- board text added: "Vehicle Control Unit LHRs Jacob Guidry Tony Chen"
- board text removed: "CAN_BREAKOUT"

Commit message: is it time to give up :3
Parts:
- removed D9: D, Active-PrechargeLib:SODFL4724X108N
- removed the G*** at (149.3, 121.0)
- removed J16: Conn_01x08, Connector_PinHeader_2.54mm:PinHeader_1x08_P2.54mm_Vertical
- removed LV4, LV5: LED, LED_SMD:LED_0805_2012Metric
- added C17: 0.1u, Capacitor_SMD:C_0805_2012Metric, F.Cu at (159.8, 68.4)
- added LED3: LED, LED_SMD:LED_0805_2012Metric, F.Cu at (176.8, 73.4)
- added LED4: LED, LED_SMD:LED_0805_2012Metric, F.Cu at (179.1, 73.4)
- C10: value 10u -> 0.1u; footprint Capacitor_SMD:C_0603_1608Metric -> Capacitor_SMD:C_0805_2012Metric
- C11: value 1u -> 10u
- C12, C14, C6: value 0.1u -> 1u
- C13: value 1u -> 0.1u
- C3, C7: value 1u -> 0.1u; footprint Capacitor_SMD:C_0603_1608Metric -> Capacitor_SMD:C_0805_2012Metric
- C4, C5: footprint Capacitor_SMD:C_0603_1608Metric -> Capacitor_SMD:C_0805_2012Metric
- C8: value 10u -> 1u
- C9: value 0.1u -> 10u; footprint Capacitor_SMD:C_0603_1608Metric -> Capacitor_SMD:C_0805_2012Metric
- D2, D3: footprint LED_SMD:LED_0603_1608Metric -> LED_SMD:LED_0805_2012Metric
- D5: value TVS -> PRTR5V0U2AX,215; footprint Diode_SMD:D_0603_1608Metric -> tv diode:PRTR5V0U2X
- D7: value TVS -> D; footprint Diode_SMD:D_0603_1608Metric -> Active-PrechargeLib:SODFL4724X108N
- J10: value CAR_CAN_Breakout -> USB_C_Receptacle_USB2.0_16P; footprint Connector_PinHeader_2.54mm:PinHeader_1x02_P2.54mm_Vertical -> USBC:GCT_USB4215-03-A_REVA
- J11: value USB_C_Receptacle_USB2.0_16P -> UART_Breakout; footprint USBC:GCT_USB4215-03-A_REVA -> Connector_PinHeader_2.54mm:PinHeader_1x02_P2.54mm_Vertical
- J12: value UART_Breakout -> Conn_01x04; footprint Connector_PinHeader_2.54mm:PinHeader_1x02_P2.54mm_Vertical -> utsvt_conn:Molex_MicroFit3.0_1x4xP3.00mm_PolarizingPeg_Vertical
- J14: footprint utsvt_conn:Molex_MicroFit3.0_1x4xP3.00mm_PolarizingPeg_Vertical -> Connector_PinHeader_2.54mm:PinHeader_1x04_P2.54mm_Vertical
- J15: value Conn_01x04 -> Conn_01x08; footprint Connector_PinHeader_2.54mm:PinHeader_1x04_P2.54mm_Vertical -> Connector_PinHeader_2.54mm:PinHeader_1x08_P2.54mm_Vertical
- J4: value Precharge+_Conn -> Conn_01x02
- J5: value Precharge-_Conn -> Conn_01x02
- J6: value Conn_02x04_Counter_Clockwise -> Conn_01x04; footprint utsvt_conn:Molex_MicroFit3.0_2x4xP3.00mm_PolarizingPeg_Vertical -> Connector_Molex:Molex_Nano-Fit_105309-xx04_1x04_P2.50mm_Vertical
- J7: value MOTOR_CAN_Breakout -> Conn_01x04; footprint Connector_PinHeader_2.54mm:PinHeader_1x02_P2.54mm_Vertical -> Connector_Molex:Molex_Nano-Fit_105309-xx04_1x04_P2.50mm_Vertical
- J8: value CAR_CAN_IN -> MOTOR_CAN_Breakout; footprint Connector_Molex:Molex_Nano-Fit_105309-xx02_1x02_P2.50mm_Vertical -> Connector_PinHeader_2.54mm:PinHeader_1x02_P2.54mm_Vertical
- J9: value CAR_CAN_OUT -> CAR_CAN_Breakout; footprint Connector_Molex:Molex_Nano-Fit_105309-xx02_1x02_P2.50mm_Vertical -> Connector_PinHeader_2.54mm:PinHeader_1x02_P2.54mm_Vertical
- moved J1 93.0 mm to (138.4, 46.2)
- moved H2 90.0 mm to (190.8, 46.9)
- moved Q1 81.4 mm to (141.5, 52.1), turned to 90 degrees
- moved R4 79.8 mm to (147.3, 52.9), turned to 0 degrees
- moved LV1 79.7 mm to (151.3, 52.9), turned to 180 degrees
- moved J8 77.5 mm to (176.4, 58.3), turned to 180 degrees
- moved J4 76.7 mm to (165.8, 45.3), turned to 90 degrees
- moved C2 75.3 mm to (147.3, 55.1), turned to 0 degrees
- moved R1 72.8 mm to (137.5, 57.6), turned to 0 degrees
- moved J5 71.9 mm to (156.2, 45.4), turned to 90 degrees
- moved J9 71.5 mm to (176.5, 64.8), turned to 180 degrees
- moved D1 70.4 mm to (142.1, 57.6), turned to 180 degrees
- moved G*** 67.1 mm to (178.7, 118.2)
- moved C15 65.0 mm to (119.5, 76.2), turned to 0 degrees
- moved D7 59.6 mm to (124.9, 64.5), turned to 180 degrees
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- renumbered LV2 to LED1, LV3 to LED2
Connections:
- C10 pad 1: /ESP/5V_USB -> /ESP/3V3
- C11 pad 1: GND -> /ESP/5V_USB
- C11 pad 2: /M_Sense -> GND
- C12 pad 1: Net-(J13-Pin_2) -> GND
- C12 pad 2: GND -> /M_Sense
- C13 pad 1: GND -> Net-(J12-Pin_2)
- C13 pad 2: /MPre_Sense -> GND
- C14 pad 1: Net-(J14-Pin_2) -> GND
- C14 pad 2: GND -> /MPre_Sense
- C15 pad 1: /ESP/RESET -> Net-(J13-Pin_2)
- C16 pad 1: /ESP/BOOT -> /ESP/RESET
- C3 pad 1: 3V3_LSOM -> +12V
- C4 pad 1: /ESP/5V_USB -> 3V3_LSOM
- C5 pad 1: /ESP/3V3_USB -> /ESP/5V_USB
- C6 pad 1: /ESP/3V3 -> /ESP/3V3_USB
- C7 pad 1: /ESP/3V3_USB -> /ESP/3V3
- C8 pad 1: /ESP/3V3 -> /ESP/3V3_USB
- D5 pad 2: /ESP/VBUSB -> /ESP/USB_D-
- D6 pad 2: /ESP/USB_D- -> /ESP/VBUSB
- D7 pad 1: GND -> +12V
- D7 pad 2: /ESP/USB_D+ -> /ContactorDriver/MCon-
- D8 pad 2: /ContactorDriver/MCon- -> /ContactorDriver/M_PreCon-
- J12 pad 1: /ESP_TX -> /ContactorDriver/MCon-
- J12 pad 2: /ESP_RX -> Net-(J12-Pin_2)
- J13 pad 1: /ContactorDriver/MCon- -> /ContactorDriver/M_PreCon-
- J14 pad 1: /ContactorDriver/M_PreCon- -> /ESP/IO1
- J14 pad 2: Net-(J14-Pin_2) -> /ESP/IO2
- J14 pad 3: +12V -> /ESP/IO3
- J14 pad 4: +12V -> /ESP/IO4
- J15 pad 1: /ESP/IO1 -> /ESP/IO5
- J15 pad 2: /ESP/IO2 -> /ESP/IO6
- J15 pad 3: /ESP/IO3 -> /ESP/IO7
- J15 pad 4: /ESP/IO4 -> /ESP/IO8
- J3 pad 41: /LED2 -> /LED4
- J3 pad 42: /LED4 -> /LED2
- J3 pad 43: /LED1 -> /LED3
- J3 pad 44: /LED3 -> /LED1
- J4 pad 1: /VPrecharge+ -> /ISO_ADC_CLK
- J4 pad 2: /ISO_ADC_CLK -> /VPrecharge+
- J5 pad 1: /VPrecharge- -> /ISO_ADC_CLK
- J5 pad 2: /ISO_ADC_CLK -> /VPrecharge-
- J6 pad 1: +12V -> /C_CAN_L
- J6 pad 2: GND -> /C_CAN_H
- J6 pad 3: /M_CAN_H -> /C_CAN_L
- J6 pad 4: /M_CAN_L -> /C_CAN_H
- J7 pad 1: /M_CAN_H -> /M_CAN_L
- J7 pad 2: /M_CAN_L -> /M_CAN_H
- J8 pad 1: /C_CAN_H -> /M_CAN_H
- J8 pad 2: /C_CAN_L -> /M_CAN_L
- R17 pad 1: Net-(J13-Pin_2) -> Net-(J12-Pin_2)
- R22 pad 1: Net-(J14-Pin_2) -> Net-(J13-Pin_2)
- U3 pad 23: /ESP/BOOT -> /ESP/LED3
- U3 pad 24: /ESP/LED3 -> /ESP/BOOT
Routing:
- net 3V3_LSOM: track 31.8 -> 111.5 mm
- net GND: track 6.20 -> 73.9 mm, vias 178 -> 71
- net /M_CAN_L: track 37.5 -> 91.1 mm, vias 0 -> 2
- net /M_CAN_H: track 37.5 -> 90.7 mm, vias 1 -> 2
- net /LED4: track 11.9 -> 49.7 mm, vias 0 -> 2
- net /LED3: track 11.3 -> 47.9 mm, vias 0 -> 2
- net /ESP/BOOT: track 56.4 -> 88.6 mm, vias 3 -> 4
- net /LED2: track 18.2 -> 50.1 mm
- net /LED1: track 17.6 -> 47.5 mm
- net /ESP/RESET: track 66.6 -> 92.8 mm, vias 2 -> 4
- net /VPrecharge-: track 45.4 -> 70.0 mm, vias 1 -> 0
- net /ISO_ADC_CLK: track 55.5 -> 78.5 mm
- net +12V: track 21.5 -> 0.47 mm, vias 9 -> 24
- net /M_Enable: track 49.4 -> 70.0 mm
- net /C_CAN_L: track 71.7 -> 90.5 mm
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- added copper zone on B.Cu, net +12V
- added copper zone on F.Cu, net +12V
- added copper zone on F.Cu, net /ContactorDriver/MCon-
- added copper zone on F.Cu, net /ContactorDriver/M_PreCon-
- added copper zone on F.Cu, net /LV+
- added copper zone on F.Cu, net 3V3_LSOM
- removed copper zone on In2.Cu, net +12V
- removed copper zone on B.Cu, net 3V3_LSOM
- removed copper zone on In1.Cu, net GND
- removed copper zone on In2.Cu, net GND
Other:
- outline, holes or cut-outs redrawn
- copper layers 4 -> 2
- board text added: "C_CAN_H C_CAN_L"
- board text added: "M_CAN_H M_CAN_L"
- board text added: "Vehicle Control Unit Rev. A 2025 LHRs Jacob Guidry Tony Chen"
- board text removed: "CAN_H"
- board text removed: "CAN_L"
- board text removed: "CAN_L CAN_H"
- board text removed: "CAR_CAN_BREAKOUT"
- board text removed: "MOTOR CAN_BREAKOUT"
- board text removed: "Vehicle Control Unit LHRs Jacob Guidry Tony Chen"

Commit message: minor fixes
Parts:
- removed LV6, LV7, LV8, LV9: LED, LED_SMD:LED_0805_2012Metric
- added G***: LOGO, LOGO, F.Cu at (153.6, 77.2)
- added G***: LOGO, UTSVT_Special:Hallock_Image_Tiny, B.Cu at (185.3, 107.0)
- added LV2: LED, LED_SMD:LED_0805_2012Metric, F.Cu at (136.6, 93.0)
- added LV3: LED, LED_SMD:LED_0805_2012Metric, F.Cu at (134.3, 93.0)
- added LV4: LED, LED_SMD:LED_0805_2012Metric, F.Cu at (132.1, 93.0)
- added LVPWR1: LED, LED_SMD:LED_0805_2012Metric, F.Cu at (151.3, 52.8)
- moved G*** 51.8 mm to (185.3, 105.6)
- moved LV1 42.1 mm to (138.8, 93.0), turned to -90 degrees
- moved G*** 30.8 mm to (169.5, 108.5)
- moved LVGND_TP1 14.5 mm to (144.1, 90.0)
- moved R27 8.52 mm to (138.8, 96.5)
- moved R28 8.52 mm to (136.6, 96.5)
- moved R29 8.52 mm to (134.3, 96.5)
- moved R30 8.27 mm to (132.1, 96.5)
- moved R26 7.64 mm to (160.5, 61.4), turned to 0 degrees
- moved C17 4.91 mm to (160.5, 63.5), turned to 180 degrees
- moved R25 3.38 mm to (144.8, 65.3), turned to 0 degrees
- moved G*** 2.34 mm to (175.9, 92.4)
- moved C16 1.07 mm to (144.8, 67.5), turned to 180 degrees
- moved 12V_TP1 0.51 mm to (145.5, 60.9)
Connections:
- R27 pad 2: Net-(LV6-A) -> Net-(LV1-A)
- R4 pad 2: Net-(LV1-A) -> Net-(LVPWR1-A)
- U3 pad 24: /ESP/BOOT -> /ESP/LED4
- U3 pad 25: /ESP/LED4 -> /ESP/BOOT
Routing:
- net /ESP/BOOT: track 88.6 -> 96.6 mm, vias 4 -> 6
- net /ESP/LED1: track 46.2 -> 40.1 mm
- net /ESP/LED4: track 43.3 -> 38.0 mm
- net /ESP/LED3: track 41.5 -> 38.3 mm
- net /ESP/LED2: track 41.4 -> 38.3 mm
- net /ESP/Buttons_LEDs_IO/3V3: track 14.3 -> 17.4 mm
- net Net-(LVPWR1-A): track 0.00 -> 2.10 mm
- net Net-(LV6-A): track 1.65 -> 0.00 mm
- net /MPre_Enable: track 54.5 -> 55.6 mm
- net /ESP_RX: track 77.0 -> 78.0 mm
- net /ESP_TX: track 79.1 -> 80.0 mm
- net /M_Enable: track 70.0 -> 69.4 mm
- net /ISO_ADC_CLK: track 78.5 -> 78.0 mm
- net /ESP/VBUSB: track 19.6 -> 19.7 mm, vias 4 -> 3
- net GND: vias 71 -> 168
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