File: VehicleControlUnit.kicad_pcb (KiCad board)
At the start: 2 copper layers, 86.6 x 100 mm, 105 parts, among them Con1 LED, Con2 LED, J1 Conn_01x02, J10 USB_C_Receptacle_USB2.0_16P, J11 UART_Breakout, J12 Conn_01x04, J13 Conn_01x04, J14 Conn_01x04, J15 Conn_01x08, J2 Precharge_Ready, J4 Conn_01x02, J5 Conn_01x02, J6 Conn_01x04, J7 Conn_01x04, J8 MOTOR_CAN_Breakout, J9 CAR_CAN_Breakout, Q1 Q_PMOS_GDS, Q2 IRLML0030, Q3 IRLML0030, SW1 RESET, SW2 BOOT, U1 TLV1117LV33DCYR, U3 ESP32-C6-MINI-1/U, U4 TCMT1106, U5 TCMT1106

Commit message: 24v changes
Parts:
- removed 12V_TP1: TestPoint, UTSVT_Special:TestPoint_HEX_3mmID
- removed the G*** at (185.3, 107.0)
- added 24V_TP1: TestPoint, UTSVT_Special:TestPoint_HEX_3mmID, F.Cu at (144.0, 60.8)
- added J16: Conn_01x08, Connector_PinHeader_2.54mm:PinHeader_1x08_P2.54mm_Vertical, F.Cu at (171.0, 62.0)
- Q1: value Q_PMOS_GDS -> PMV35EPER
- R17, R19, R22, R24, R4: value 2k -> 4k
- moved J8 6.29 mm to (182.7, 59.0)
- moved J9 6.29 mm to (182.8, 65.4)
- moved SW2 4.40 mm to (161.2, 68.3)
- moved LED2 4.15 mm to (178.6, 73.2)
- moved LED3 4.15 mm to (180.9, 73.2)
- moved LED4 4.15 mm to (183.2, 73.2)
- moved LED1 4.15 mm to (176.2, 73.2)
- moved R5 4.15 mm to (176.2, 76.8)
- moved R6 4.15 mm to (178.6, 76.9)
- moved R7 4.15 mm to (180.9, 76.9)
- moved R8 4.15 mm to (183.2, 76.9)
- moved LVGND_TP1 2.21 mm to (143.4, 87.9)
- moved D6 0.80 mm to (120.1, 118.0)
Connections:
- net +12V renamed +24V
- J4 pad 1: /ISO_ADC_CLK -> GND
- J5 pad 1: /ISO_ADC_CLK -> GND
- U3 pad 22: unconnected-(U3-GPIO8-Pad22) -> /ESP/LED3
- U3 pad 23: /ESP/LED3 -> /ESP/LED4
- U3 pad 24: /ESP/LED4 -> /ESP/BOOT
- U3 pad 25: /ESP/BOOT -> unconnected-(U3-GPIO19-Pad25)
Routing:
- net /ISO_ADC_CLK: track 78.0 -> 0.00 mm
- net 3V3_LSOM: track 111.8 -> 153.8 mm, vias 6 -> 8
- net /M_Enable: track 69.4 -> 109.4 mm, vias 2 -> 3
- net /Precharge_Ready: track 38.7 -> 78.5 mm, vias 0 -> 2
- net /MPre_Enable: track 55.6 -> 88.4 mm, vias 2 -> 3
- net /M_Sense: track 62.8 -> 95.2 mm, vias 2 -> 4
- net /MPre_Sense: track 58.8 -> 87.9 mm, vias 2 -> 4
- net /VPrecharge-: track 69.5 -> 76.8 mm, vias 0 -> 1
- net GND: track 73.9 -> 80.6 mm, vias 168 -> 161
- net /M_CAN_L: track 91.4 -> 84.8 mm
- net /M_CAN_H: track 90.9 -> 84.4 mm
- net /VPrecharge+: track 66.0 -> 71.9 mm
- net /C_CAN_H: track 87.5 -> 81.9 mm
- net /ESP/BOOT: track 96.6 -> 91.6 mm, vias 6 -> 4
- net /C_CAN_L: track 90.6 -> 86.4 mm
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Other:
- board text added: "MPre_Sense"
- board text added: "M_Sense"
