File: Power.kicad_sch (KiCad schematic)
At the start: 20 parts, among them IC1 LM74502HDDFR, J1 CarLVPowerConnector, J3 Conn_01x02, Q1 PSMN8R5-40MSDX

Commit message: ravi's bs
Parts:
- R1: value 4k -> 4.3k
- R13: value 8k -> 9k
Other:
- note added: "Overvoltage Protection: 29.03V Vovr = (R2 * Vov)/(R1 + R2) Vov = Vovr * (R1 + R2) / R2 29.03 = 1.25 * (200k + 9k) / 9k"
Changed lines of the file:
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@@
 	(generator_version "9.0")
 	(paper "A4")
+	(text "Overvoltage Protection: 29.03V\nVovr = (R2 * Vov)/(R1 + R2)\nVov = Vovr * (R1 + R2) / R2\n29.03 = 1.25 * (200k + 9k) / 9k"
+		(exclude_from_sim no)
+		(at 146.685 69.85 0)
+		(effects
+			(font
+				(size 1.27 1.27)
+			)
+		)
+	)
 	(text "3v3 injector"
 		(exclude_from_sim no)
@@
 			)
 		)
-		(property "Value" "4k"
+		(property "Value" "4.3k"
 			(at 193.04 41.2749 0)
 			(effects
@@
 		(fields_autoplaced yes)
 		(property "Reference" "R13"
-			(at 120.65 66.675 90)
-			(effects
-				(font
-					(size 1.27 1.27)
-				)
-			)
-		)
-		(property "Value" "8k"
-			(at 120.65 69.215 90)
-			(effects
-				(font
+			(at 120.65 66.04 90)
+			(effects
+				(font
+					(size 1.27 1.27)
+				)
+			)
+		)
+		(property "Value" "9k"
+			(at 120.65 68.58 90)
+			(effects
+				(font

Commit message: bom stuff
Parts:
- C21: value 220u -> 10u
Changed lines of the file:
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@@
 			)
 		)
-		(property "Value" "220u"
+		(property "Value" "10u"
 			(at 114.935 48.8949 0)
 			(effects
