File: Hardware/ESP.kicad_sch (KiCad schematic)
At the start: 28 parts, among them J9 USB_C_Receptacle_USB2.0_16P, U1 TPS2115ADRBR, U4 ESP32-C6-MINI-1/U, U8 LT1963AEST-3.3#TRPBF

Commit message: review council
Parts:
- 3V31: now fitted
Connections:
- net IO10: no longer names the net of U4.6 (GPIO3/ADC1_CH3)
- net IO12: no longer names the net of U4.5 (GPIO2/ADC1_CH2)
- net IO4: no longer names the net of U4.16 (MTDO/GPIO7)
- net IO5: no longer names the net of U4.15 (MTCK/GPIO6/ADC1_CH6)
- net IO6: no longer names the net of U4.13 (GPIO1/ADC1_CH1/XTAL_32K_N)
- net IO7: no longer names the net of U4.12 (GPIO0/ADC1_CH0/XTAL_32K_P)
- net IO8: no longer names the net of U4.10 (MTDI/GPIO5/ADC1_CH5)
- net IO9: no longer names the net of U4.9 (MTMS/GPIO4/ADC1_CH4)
- no-connect marks 7 -> 15
Other:
- sheet Buttons_LEDs_IO ports: added none; removed IO10, IO12, IO4, IO5, IO6, IO7, IO8, IO9
- note added: "3.3V MUX"
- note removed: "5V MUX"

Commit message: only 1 crash not bad
Parts:
- renumbered 3V31 to 3V1, C6 to C1, C8 to C2, C7 to C3, C10 to C4, C13 to C5, C12 to C6, C9 to C7, C11 to C8, D4 to D3, D1 to D4, D2 to D5, D3 to D6, D6 to D7, D9 to D8, J9 to J6, R8 to R1, R9 to R2, R10 to R3, R11 to R4, R6 to R5, R7 to R6, R29 to R7, R30 to R8, R31 to R9, U1 to U2, U8 to U3

Commit message: i hate everything about you - three days grace
Parts:
- 3V1: footprint TestPoint:TestPoint_Pad_2.0x2.0mm -> TestPoint:TestPoint_Keystone_5005-5009_Compact
Changed lines of the file:
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@@
 			)
 		)
-		(property "Footprint" "TestPoint:TestPoint_Pad_2.0x2.0mm"
+		(property "Footprint" "TestPoint:TestPoint_Keystone_5005-5009_Compact"
 			(at 96.52 27.305 0)
 			(effects

Commit message: bom, cpl, and friends
Parts:
- D3: Mouser Part Number 621-1N5819HW-F -> 621-1N5819HW-F
- R8: Mouser Part Number (none) -> 71-CRCW060310K0FKEI; P/N (none) -> CRCW060310K0FKEI
