File: Hardware/Status_LEDs.kicad_sch (KiCad schematic)
At the start: 34 parts

Commit message: only 1 crash not bad
Parts:
- added LV22: Driving, LED_SMD:LED_0603_1608Metric_Pad1.05x0.95mm_HandSolder, symbol Device:LED
- added R49: 1k, Resistor_SMD:R_0603_1608Metric_Pad0.98x0.95mm_HandSolder, symbol Device:R_US
Connections:
- net GND: now also LV22.1 (K)
- net LED1 renamed MPre_Sense
- net LED2 renamed MPre_Enable
- net LED3 renamed M_Sense
- net LED4 renamed M_Enable
- new net: LV22.2 (A), R49.2
- new net ESP_RESET: R49.1

Commit message: fixing
Parts:
- added LV23: PT, LED_SMD:LED_0603_1608Metric_Pad1.05x0.95mm_HandSolder, symbol Device:LED
- added R52: 1k, Resistor_SMD:R_0603_1608Metric_Pad0.98x0.95mm_HandSolder, symbol Device:R_US
Connections:
- net at R32.2: now also LV5.1 (K); no longer LV5.2 (A)
- net at R40.2: now also LV13.1 (K); no longer LV13.2 (A)
- net at R48.2: now also LV21.1 (K); no longer LV21.2 (A)
- net at R35.2: now also LV8.1 (K); no longer LV8.2 (A)
- net at R42.2: now also LV15.1 (K); no longer LV15.2 (A)
- net at R37.2: now also LV10.1 (K); no longer LV10.2 (A)
- net at R49.2: now also LV22.1 (K); no longer LV22.2 (A)
- net at R34.2: now also LV7.1 (K); no longer LV7.2 (A)
- net at R47.2: now also LV20.1 (K); no longer LV20.2 (A)
- net at R45.2: now also LV18.1 (K); no longer LV18.2 (A)
- net at R33.2: now also LV6.1 (K); no longer LV6.2 (A)
- net at R39.2: now also LV12.1 (K); no longer LV12.2 (A)
- net at R43.2: now also LV16.1 (K); no longer LV16.2 (A)
- net at R38.2: now also LV11.1 (K); no longer LV11.2 (A)
- net at R46.2: now also LV19.1 (K); no longer LV19.2 (A)
- net at R41.2: now also LV14.1 (K); no longer LV14.2 (A)
- net at R44.2: now also LV17.1 (K); no longer LV17.2 (A)
- net at R36.2: now also LV9.1 (K); no longer LV9.2 (A)
- removed net GND: LV10.1 (K), LV11.1 (K), LV12.1 (K), LV13.1 (K), LV14.1 (K), LV15.1 (K), LV16.1 (K), LV17.1 (K), LV18.1 (K), LV19.1 (K), LV20.1 (K), LV21.1 (K), LV22.1 (K), LV5.1 (K), LV6.1 (K), LV7.1 (K), LV8.1 (K), LV9.1 (K)
- net Sense_Timeout renamed PreSense_Timeout
- new net: LV23.1 (K), R52.2
- new net +3V3: LV22.2 (A)
- new net 3V3_LSOM: LV10.2 (A), LV11.2 (A), LV12.2 (A), LV13.2 (A), LV14.2 (A), LV15.2 (A), LV16.2 (A), LV17.2 (A), LV18.2 (A), LV19.2 (A), LV20.2 (A), LV21.2 (A), LV23.2 (A), LV5.2 (A), LV6.2 (A), LV7.2 (A), LV8.2 (A), LV9.2 (A)
- new net Motor_Sense_Timeout: R52.1
Other:
- moved on the sheet: LV10, LV11, LV12, LV13, LV14, LV15, LV16, LV17, LV18, LV19, LV20, LV21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
