File: Hardware/VehicleControlUnit.kicad_sch (KiCad schematic)
At the start: 14 parts, among them J10 Conn_01x04, J14 PeripheralCAN, J15 CarCANConnector, J16 CarCANConnector, J4 Conn_02x06_Counter_Clockwise, J5 SFH11-PBPC-D05-ST-BK, U6 LeaderSOM

Commit message: review council
Parts:
- removed J14: PeripheralCAN, UTSVT_Connectors:Molex_Nano-Fit_105309-xx04_1x04_P2.50mm_Vertical, symbol UTSVT_Connectors:PeripheralCANConnector
- removed J15, J16: CarCANConnector, UTSVT_Connectors:Molex_Nano-Fit_105309-xx02_1x02_P2.50mm_Vertical, symbol UTSVT_Connectors:CarCANConnector
- added J2: CarCAN, symbol Connector_Generic:Conn_01x04
- added J6: MotorCAN, symbol Connector_Generic:Conn_01x03
- H1, H2, H3, J10, LOGO1, LOGO2: now fitted
- J4: value Conn_02x06_Counter_Clockwise -> Precharge Connector
Connections:
- net Batt_Voltage: now also J10.4 (Pin_4), U6.12 (ADC1_IN11); no longer J10.3 (Pin_3), U6.43 (ADC1_IN1)
- net C_CAN_H: now also J2.2 (Pin_2), J2.4 (Pin_4)
- net C_CAN_L: now also J2.1 (Pin_1), J2.3 (Pin_3)
- net ESP_RESET: now also U6.31 (ADC1_IN12); no longer U6.10 (ADC2_IN12)
- net GND: now also J10.3 (Pin_3); no longer J10.4 (Pin_4)
- net MPre_Sense: now also U6.14 (SPI2_MISO); no longer U6.5 (I2C4_SDA)
- net M_CAN_H: now also J6.3 (Pin_3)
- net M_CAN_L: now also J6.2 (Pin_2)
- net M_Sense: now also U6.18 (SPI2_MOSI); no longer U6.11 (I2C3_SCL)
- net Motor_Voltage: now also U6.10 (ADC2_IN12); no longer U6.41 (ADC1_IN2)
- net Precharge_Complete: now reaches U6.13 (UART5_TX)
- net Precharge_Timeout: now reaches U6.15 (UART5_RX)
- net Sense_Timeout: now reaches U6.17 (USART1_TX)
- net Motor_Fault: now reaches U6.19 (USART1_RX)
- net SWOC: now reaches U6.7 (I2C4_SCL)
- net Motor_Watchdog: now reaches U6.9 (I2C3_SDA)
- net Driving: now reaches U6.45 (ADC1_IN8)
- net Safe: now reaches U6.47 (ADC1_IN6)
- net LED5 renamed HB
- new net BPS_Fault: U6.5 (I2C4_SDA)
- new net Bad_Hall: U6.11 (I2C3_SCL)
- new net Cruise: U6.43 (ADC1_IN1)
- new net Regen: U6.41 (ADC1_IN2)
- no-connect marks 18 -> 5
Other:
- added sheet Status LEDs (Status_LEDs.kicad_sch)

Commit message: only 1 crash not bad
Parts:
- added C21, C22: 0.1u, Capacitor_SMD:C_0603_1608Metric_Pad1.08x0.95mm_HandSolder, symbol Device:C
- added R50, R51: 1k, Resistor_SMD:R_0603_1608Metric_Pad0.98x0.95mm_HandSolder, symbol Device:R_US
- J3: renamed from J10; value Conn_01x04 -> 3.3V Injector
- J4: renamed from J2; footprint (none) -> UTSVT_Connectors:Molex_Nano-Fit_105309-xx04_1x04_P2.50mm_Vertical
- J5: renamed from J6; footprint (none) -> Connector_Molex:Molex_Nano-Fit_105309-xx03_1x03_P2.50mm_Vertical
- renumbered D10 to D1, D11 to D2, J4 to J1, J5 to J2, U6 to U1
Connections:
- net LED1 is gone; now on net Driving: U1.48 (SPI3_SCK)
- net LED2 is gone; now on net Cruise: U1.46 (SPI3_MOSI)
- net LED3 is gone; now on net Regen: U1.44 (SPI3_NSS)
- net LED4 is gone; now on net HB: U1.42 (SPI3_MISO)
- net Batt_Voltage: now also J3.2 (Pin_2), U1.10 (ADC2_IN12), C22.2, R51.1; no longer D1.1 (K), J1.7 (Pin_7), J3.4 (Pin_4), U1.12 (ADC1_IN11)
- net Cruise: no longer U1.43 (ADC1_IN1)
- net Driving: no longer U1.45 (ADC1_IN8)
- net ESP_RESET: no longer J2.5 (CH5)
- net ESP_RX: now also J2.9 (CH1); no longer J2.3 (CH7)
- net ESP_TX: now also J2.10 (CH0); no longer J2.4 (CH6)
- net GND: now also C21.1, C22.1
- net HB: no longer U1.40 (ADC1_IN7)
- net MPre_Enable: no longer J2.7 (CH3)
- net MPre_Sense: no longer J2.6 (CH4)
- net M_Enable: no longer J2.9 (CH1)
- net M_Sense: no longer J2.8 (CH2)
- net Motor_Voltage: now also J3.4 (Pin_4), U1.12 (ADC1_IN11), C21.2, R50.1; no longer D2.1 (K), J1.12 (Pin_12), J3.2 (Pin_2), U1.10 (ADC2_IN12)
- net Regen: no longer U1.41 (ADC1_IN2)
- new net B_Volt: D1.1 (K), J1.7 (Pin_7), R51.2
- new net M_Volt: D2.1 (K), J1.12 (Pin_12), R50.2
- no-connect marks 5 -> 14
Other:
- sheet Status LEDs ports: added {Status_LEDs}; removed {Status_LEDS}

Commit message: fixing
Parts:
- H1, H2, H3: footprint MountingHole:MountingHole_3.2mm_M3 -> MountingHole:MountingHole_3.2mm_M3_Pad_TopBottom; symbol Mechanical:MountingHole -> Mechanical:MountingHole_Pad
Connections:
- net Sense_Timeout is gone; now on net MPre_Enable: U1.17 (USART1_TX)
- net BPS_Fault: now also U1.16 (SPI2_NSS); no longer U1.5 (I2C4_SDA)
- net Bad_Hall: now also U1.48 (SPI3_SCK); no longer U1.11 (I2C3_SCL)
- net Cruise: now also U1.20 (SPI2_SCK); no longer U1.46 (SPI3_MOSI)
- net Driving: now also U1.9 (I2C3_SDA); no longer U1.48 (SPI3_SCK)
- net HB: now also U1.14 (SPI2_MISO); no longer U1.42 (SPI3_MISO)
- net MPre_Enable: no longer U1.16 (SPI2_NSS)
- net MPre_Sense: now also U1.19 (USART1_RX); no longer U1.14 (SPI2_MISO)
- net M_Enable: now also U1.47 (ADC1_IN6); no longer U1.20 (SPI2_SCK)
- net M_Sense: now also U1.45 (ADC1_IN8); no longer U1.18 (SPI2_MOSI)
- net Motor_Fault: now also U1.42 (SPI3_MISO); no longer U1.19 (USART1_RX)
- net Motor_Watchdog: now also U1.46 (SPI3_MOSI); no longer U1.9 (I2C3_SDA)
- net Precharge_Complete: now also U1.11 (I2C3_SCL); no longer U1.13 (UART5_TX)
- net Regen: now also U1.18 (SPI2_MOSI); no longer U1.44 (SPI3_NSS)
- net SWOC: now also U1.44 (SPI3_NSS); no longer U1.7 (I2C4_SCL)
- net Safe: now also U1.7 (I2C4_SCL); no longer U1.47 (ADC1_IN6)
- new net Motor_Sense_Timeout: U1.5 (I2C4_SDA)
- new net PreSense_Timeout: U1.13 (UART5_TX)
- no-connect marks 14 -> 16
Other:
- moved on the sheet: J2, J3

Commit message: added connector models
Parts:
- J1: footprint Connector_Molex:Molex_Nano-Fit_105310-xx12_2x06_P2.50mm_Vertical -> UTSVT_Connectors:Molex_Nano-Fit_105310-xx12_2x06_P2.50mm_Vertical
- J5: footprint Connector_Molex:Molex_Nano-Fit_105309-xx03_1x03_P2.50mm_Vertical -> UTSVT_Connectors:Molex_Nano-Fit_105309-xx03_1x03_P2.50mm_Vertical
Changed lines of the file:
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@@
 			)
 		)
-		(property "Footprint" "Connector_Molex:Molex_Nano-Fit_105309-xx03_1x03_P2.50mm_Vertical"
+		(property "Footprint" "UTSVT_Connectors:Molex_Nano-Fit_105309-xx03_1x03_P2.50mm_Vertical"
 			(at 248.285 52.07 0)
 			(effects
@@
 			)
 		)
-		(property "Footprint" "Connector_Molex:Molex_Nano-Fit_105310-xx12_2x06_P2.50mm_Vertical"
+		(property "Footprint" "UTSVT_Connectors:Molex_Nano-Fit_105310-xx12_2x06_P2.50mm_Vertical"
 			(at 51.435 165.1 0)
 			(effects

Commit message: bom, cpl, and friends
Parts:
- J1: Mouser Part Number (none) -> 538-105310-1112; P/N (none) -> 105310-1112
- J4: Mouser Part Number (none) -> 538-105309-1104; P/N (none) -> 105309-1104
- J5: Mouser Part Number (none) -> 538-105309-1103; P/N (none) -> 105309-1103
- U1: now left out of the parts list
