File: Hardware/VehicleControlUnit/VehicleControlUnit.kicad_sch (KiCad schematic)
At the start: 0 parts

Commit message: lil shah getting touche' (with accent on e)
Other:
- added sheet 12VBuck (12VBuck.kicad_sch)
- added sheet 5VBuck (5VBuck.kicad_sch)
- added sheet CAN_Transceiver (CAN_Transceiver.kicad_sch)
- added sheet ESP32 (ESP32.kicad_sch)
- added sheet LDO (LDO.kicad_sch)
